File: rover-chasis-controller.kicad_sch (KiCad schematic)
At the start: 88 parts, among them J1 Screw_Terminal_01x02, J10 GPS Interface, J11 Compass Connection (I2C), J12 External LED (Red), J13 External LED (Yellow), J14 External LED (Green), J2 Motor control, J3 Encoder, J4 External LED, J5 External LED, J6 External LED, J7 TTL, J8 Ultrasonic Sensor Inputs, J9 MPU-6050 IMU Module, Q1 IRF9540N, Q10 MMPQ3904, Q11 MMPQ3904, Q12 MMPQ3904, Q2 NPN, Q3 NPN, Q4 NPN, Q5 NPN, Q6 MMPQ3904, Q7 NPN, Q8 NPN, Q9 NPN, U1 LD1117S33TR_SOT223, U3 TPS5430DDA

Commit message: Issue #1: Major revision
Parts:
- removed Q12: MMPQ3904, easyeda2kicad:SOIC-16_L9.9-W3.9-P1.27-LS6.0-BL, symbol C904282:MMPQ3904
- added BZ2: Buzzer, symbol Device:Buzzer
- added C21, C22, C23, C24, C25, C26, C27, C28, C29, C30, C31, C32, C35, C36, C47, C49: 0.1 uF, symbol Device:C
- added C33, C34, C37, C38: 10 uF, symbol Device:C
- added C39, C53: 10uF, Capacitor_SMD:C_2220_5750Metric, symbol Device:C
- added C40, C55: 2.7nF, Capacitor_SMD:C_0805_2012Metric, symbol Device:C
- added C41, C54: 100nF, Capacitor_SMD:C_0805_2012Metric, symbol Device:C
- added C42, C56: 39pF, Capacitor_SMD:C_0805_2012Metric, symbol Device:C
- added C43, C57: 47pF, Capacitor_SMD:C_0805_2012Metric, symbol Device:C
- added C44, C45, C46, C58, C59, C60: 22 uF, Capacitor_SMD:C_2220_5750Metric, symbol Device:C
- added D10, D8: SMF5V0A, Diode_SMD:D_SMF, symbol Diode:SMF5V0A
- added D11: SMAJ5.0A, Diode_SMD:D_SMA, symbol Diode:SMAJ5.0A
- added D7: D, symbol Device:D
- added F2, F3, F4: Fuse, symbol Device:Fuse
- added J15: External LED (Red), symbol Connector_Generic:Conn_01x02
- added J16: External LED (Yellow), symbol Connector_Generic:Conn_01x02
- added J17: External LED (Green), symbol Connector_Generic:Conn_01x02
- added J18, J19, J20, J21: Motor control, symbol Connector_Generic:Conn_01x04
- added J22, J23, J24: Encoder, symbol Connector_Generic:Conn_01x04
- added J25: MPU-6050 IMU Module, symbol Connector_Generic:Conn_01x04
- added J26: Screw_Terminal_01x02, symbol Connector:Screw_Terminal_01x02
- added J28: Conn_01x06, symbol Connector_Generic:Conn_01x06
- added L2, L4: 4.7uH, YSPI0724-4R7M:IND-SMD_L7.3-W6.6_YSPI07XX, symbol Device:L
- added Q12, Q15: SUD50P10-43L-TP, Package_TO_SOT_SMD:TO-252-2, symbol Transistor_FET:SUD50P10-43L
- added Q13: MMPQ3904, easyeda2kicad:SOIC-16_L9.9-W3.9-P1.27-LS6.0-BL, symbol C904282:MMPQ3904
- added R30, R31, R32, R33, R34, R35, R36, R37, R38, R39, R40, R41, R42, R43, R44, R45: 1 kO, symbol Device:R_US
- added R46, R47, R48, R49, R50, R51, R52, R53, R54, R55, R56, R57, R58, R59, R60, R61, R62, R63, R76: 10 kO, symbol Device:R_US
- added R64: 47k, Resistor_SMD:R_0805_2012Metric, symbol Device:R
- added R65: 200k, Resistor_SMD:R_0805_2012Metric, symbol Device:R
- added R66: 16k, Resistor_SMD:R_0805_2012Metric, symbol Device:R
- added R67: 120k, Resistor_SMD:R_0805_2012Metric, symbol Device:R
- added R68: 22.1k, Resistor_SMD:R_0805_2012Metric, symbol Device:R
- added R69, R70: 4.3 kO, symbol Device:R_US
- added R75: 47 kO, symbol Device:R_US
- added R77: 47 kO T+-1%, symbol Device:R_US
- added R78: 200 kO, symbol Device:R_US
- added R79: 16 kO, symbol Device:R_US
- added R80: 120 kO, symbol Device:R_US
- added R81: 22.1kO, symbol Device:R_US
- added U2: AP64500, ultralibAP64500:AP64500SP-13, symbol dcdc-lib:AP64500
- added U6: AP64500SP-13, easyeda2kicad:SO-8_L4.9-W3.9-P1.27-LS6.0-BL-EP, symbol C2070920:AP64500SP-13
- C10: value 10 uF -> 0.1 uF; LCSC https://www.lcsc.com/product-detail/Aluminum-Electrolytic-C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 -> https://www.lcsc.com/product-detail/Through-Hole-Ceramic-Ca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
Connections:
- net ADC: now also D11.1 (A1), R76.2, R77.1
- net GND: now also Q10.10 (E4), Q10.12 (E3), Q10.14 (E2), Q10.16 (E1), Q11.10 (E4), Q11.12 (E3), Q11.14 (E2), Q11.16 (E1), Q6.10 (E4), Q6.12 (E3), Q6.14 (E2), Q6.16 (E1), C21.1, C22.1, C23.1, C24.1, C25.1, C26.1, C27.1, C28.1, C29.1, C30.1, C31.1, C32.1, C33.1, C34.1, C35.1, C36.1, C37.1, C38.1, C39.2, C40.2, C42.2, C44.2, C45.2, C46.2, C47.1, C49.1, C53.2, C55.2, C56.2, C58.2, C59.2, C60.2, D10.1 (A1), D11.2 (A2), D8.1 (A1), J15.2 (Pin_2), J16.2 (Pin_2), J17.2 (Pin_2), J18.4 (Pin_4), J19.4 (Pin_4), J20.4 (Pin_4), J21.4 (Pin_4), J22.4 (Pin_4), J23.4 (Pin_4), J24.4 (Pin_4), J25.4 (Pin_4), J26.2 (Pin_2), J28.6 (Pin_6), Q13.10 (E4), Q13.12 (E3), Q13.14 (E2), Q13.16 (E1), R64.2, R65.2, R68.2, R75.2, R76.1, R78.2, R81.2, U2.7 (GND), U6.7 (GND)
- net STM32 GPIO: now also J22.1 (Pin_1), J22.2 (Pin_2), J23.1 (Pin_1), J23.2 (Pin_2), J24.1 (Pin_1), J24.2 (Pin_2), J28.1 (Pin_1), J28.2 (Pin_2), J28.3 (Pin_3), J28.4 (Pin_4), R30.1, R31.1, R32.1, R33.1, R34.1, R35.1, R36.1, R37.1, R38.1, R39.1, R40.1, R41.1, R42.1, R43.1, R44.1, R45.1, R58.1, R59.1, R60.1, R61.1, R62.1, R63.1
- net STM32 I2C: now also J25.1 (Pin_1), J25.2 (Pin_2), R69.1, R70.1
- net VCC: now also Q12.2 (D)
- net VCC (3V): now also BZ2.1 (+), C47.2, C49.2, D7.1 (K), J25.3 (Pin_3), J28.5 (Pin_5), R58.2, R59.2, R60.2, R61.2, R62.2, R63.2, R69.2, R70.2
- net VCC (5V): now also C33.2, C34.2, C35.2, C36.2, C37.2, C38.2, F2.2, F3.2, F4.2, R46.2, R47.2, R48.2, R49.2, R50.2, R51.2, R52.2, R53.2, R54.2, R55.2, R56.2, R57.2
- net Motor_PWM_Collector_4: now reaches Q10.1 (C1)
- net Motor_PWM_Collector_4: now also Q10.2 (C1), C28.2, J21.3 (Pin_3), R53.1
- net at Q10.11 (B3): now also R40.2
- net at Q10.13 (B2): now also R39.2
- net at Q10.15 (B1): now also R38.2
- net Motor_F_Collector_4: now reaches Q10.3 (C2)
- net Motor_F_Collector_4: now also Q10.4 (C2), C30.2, J21.2 (Pin_2), R55.1
- net Motor_R_Collector_4: now reaches Q10.5 (C3)
- net Motor_R_Collector_4: now also Q10.6 (C3), C32.2, J21.1 (Pin_1), R57.1
- net External_LED_Collector_3: now reaches Q10.7 (C4)
- net External_LED_Collector_3: now also Q10.8 (C4), J17.1 (Pin_1)
- net at Q10.9 (B4): now also R41.2
- net Motor_PWM_Collector_1: now reaches Q6.1 (C1)
- net Motor_PWM_Collector_1: now also Q6.2 (C1), C21.2, J18.3 (Pin_3), R46.1
- net at Q6.11 (B3): now also R31.2
- net at Q6.13 (B2): now also R32.2
- net at Q6.15 (B1): now also R33.2
- net Motor_F_Collector_1: now reaches Q6.3 (C2)
- net Motor_F_Collector_1: now also Q6.4 (C2), C23.2, J18.2 (Pin_2), R48.1
- net Motor_R_Collector_1: now reaches Q6.5 (C3)
- net Motor_R_Collector_1: now also Q6.6 (C3), C25.2, J18.1 (Pin_1), R50.1
- net Buzzer_Collector: now reaches Q6.7 (C4)
- net Buzzer_Collector: now also Q6.8 (C4), BZ2.2 (-), D7.2 (A)
- net at Q6.9 (B4): now also R30.2
- net Motor_PWM_Collector_3: now reaches Q11.1 (C1)
- net Motor_PWM_Collector_3: now also Q11.2 (C1), C22.2, J19.3 (Pin_3), R47.1
- net at Q11.11 (B3): now also R44.2
- net at Q11.13 (B2): now also R43.2
- net at Q11.15 (B1): now also R42.2
- net Motor_F_Collector_3: now reaches Q11.3 (C2)
- net Motor_F_Collector_3: now also Q11.4 (C2), C24.2, J19.2 (Pin_2), R49.1
- net Motor_R_Collector_3: now reaches Q11.5 (C3)
- net Motor_R_Collector_3: now also Q11.6 (C3), C26.2, J19.1 (Pin_1), R51.1
- net External_LED_Collector_2: now reaches Q11.7 (C4)
- net External_LED_Collector_2: now also Q11.8 (C4), J16.1 (Pin_1)
- net at Q11.9 (B4): now also R45.2
- new net: Q13.13 (B2), R35.2
- new net: C40.1, R66.2
- new net: Q13.15 (B1), R34.2
- new net: Q13.9 (B4), R37.2
- new net: C42.1, R66.1, U2.6 (COMP)
- new net: C55.1, R79.2
- new net: Q12.1 (G), R64.1
- new net: C57.2, R80.2, R81.1, U6.6 (COMP)
- new net: C43.2, R67.2, R68.1, U2.5 (FB)
- new net: C56.1, R79.1, U6.5 (FB)
- new net: C54.1, U6.1 (BST)
- new net: C53.1, Q15.3 (S), R77.2, U6.2 (VIN), U6.3 (EN)
- new net: R78.1, U6.4 (RT/CLK)
- new net: C54.2, L4.1, U6.8 (SW)
- new net: R65.1, U2.4 (RT/CLK)
- new net: F4.1, J24.3 (Pin_3)
- new net: J26.1 (Pin_1), Q15.2 (D)
- new net: F3.1, J23.3 (Pin_3)
- new net: Q15.1 (G), R75.1
- new net: Q13.11 (B3), R36.2
- new net: C41.1, U2.1 (BST)
- new net: C41.2, L2.1, U2.8 (SW)
- new net: C39.1, Q12.3 (S), U2.2 (VIN), U2.3 (EN)
- new net: F2.1, J22.3 (Pin_3)
- new net +5VD: C43.1, C44.1, C45.1, C46.1, C57.1, C58.1, C59.1, C60.1, D10.2 (A2), D8.2 (A2), L2.2, L4.2, R67.1, R80.1
- new net External_LED_Collector_1: J15.1 (Pin_1), Q13.7 (C4), Q13.8 (C4)
- new net Motor_F_Collector_2: C29.2, J20.2 (Pin_2), Q13.3 (C2), Q13.4 (C2), R54.1
- new net Motor_PWM_Collector_2: C27.2, J20.3 (Pin_3), Q13.1 (C1), Q13.2 (C1), R52.1
- new net Motor_R_Collector_2: C31.2, J20.1 (Pin_1), Q13.5 (C3), Q13.6 (C3), R56.1
- new net idk, mb some false pin: U6.9 (EP)
Other:
- note added: "4X"
- note added: "Buzzer (deprecated design)"
- note added: "CS"
- note added: "Encoders (4X)"
- note added: "I calculated value of R4, C4, R3 using formula in AP64500 doc."
- note added: "Input voltage regulator"
- note added: "LIS3DSH (I2C) (Accelerometer STM32)"
- note added: "LIS3DSH (SPI) (Accelerometer STM32)"
- note added: "MISO"
- note added: "MOSI"
- note added: "MPU-6050 IMU Module (deprecated design)"
- note added: "Motion sensor (STM32F4 user manual) The ST-MEMS motion sensor is an ultra-compact low-power three-axis linear accelerometer. The motion sensor includes a sensing element and an IC interface able to provide the measured acceleration to the external world through the I2C/SPI serial interfaces. The STM32F407VG microcontroller controls this motion sensor through the SPI interface"
- note added: "Motor controller (deprecated design)"
- note added: "Motors controllers (4X)"
- note added: "Power Supply"
- note added: "SCK"
- note added: "TODO: 4. Replace all Through-a-hole/Leaded elements with SMD. 7. Resolve all ERC exceptions and warnings. 9. Recalculate all of the numerical values for scheme, to be sure. 10. Integrate Resistor/(Capacitors) Networks, Arrays? DONE: 1. Rework transisor schemes with transistor arrays. => DONE 1.1 Motor controllers. => DONE 1.2 External LEDs. => DONE 1.3 Buzzer. => DONE 2. Rework power supply by ta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"
- note added: "Transistors Connections (4X)"
- note added: "Two options of LIS3DSH connection."
- note added: "but it can be 5V also"
- note added: "collector has two pins for better current handling and thermal dissipation"
- note added: "maybe interrupt pins: INT1/DRDY, INT2 (if we want to use interrupts)."
- note added: "maybe, bypass capacitors for noise reducing"
- note removed: "Encoder"
- note removed: "MPU-6050 IMU Module"
- note removed: "Motor controller"
- note removed: "TODO: 1. Rework transisor schemes with transistor arrays. 1.1 Motor controllers 1.2 External LEDs 1.3 Buzzer 2. Rework power supply by taking already in use PMIC in rpi-power-HAT. (Varya PCB) 3. Find out about accelerometer in STM32 instead of MPU-6050 IMU Module. 4. Replace all Through-a-hole/Leaded elements with SMD. 5. Maybe, consider TVS diode for the ADC. 6. Maybe, organize everything to dif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"
- note removed: "Transistors Connections(to be done)"
- moved on the sheet: BZ1, C15, C16, C17, C18, C19, C20, C7, C8, C9, D2, D3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

Commit message: Issue #1: Resistor arrays and refactoring
Parts:
- removed R30, R31, R32, R33, R34, R35, R36, R37, R42, R43, R44, R45: 1 kO, symbol Device:R_US
- added Q16: MMPQ3904, easyeda2kicad:SOIC-16_L9.9-W3.9-P1.27-LS6.0-BL, symbol C904282:MMPQ3904
- added RN1: 4D03WGJ0102T5E (10k), easyeda2kicad:RES-ARRAY-SMD_0603-8P-L3.2-W1.6-BL, symbol C20197:4D03WGJ0102T5E
- added RN2, RN3, RN4, RN5: 4D03WGJ0102T5E (1k), easyeda2kicad:RES-ARRAY-SMD_0603-8P-L3.2-W1.6-BL, symbol C20197:4D03WGJ0102T5E
- C10, C15, C16, C17, C20, C21, C22, C23, C24, C25, C26, C27, C28, C29, C30, C31, C32, C36, C49: value 0.1 uF -> 0.1uF
- C11, C35: value 0.1 uF -> 10uF; LCSC https://www.lcsc.com/product-detail/Through-Hole-Ceramic-Ca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 -> https://www.lcsc.com/product-detail/Aluminum-Electrolytic-C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
- C18, C19, C37: value 10 uF -> 10uF
- C34: value 10 uF -> 0.1 uF; LCSC https://www.lcsc.com/product-detail/Aluminum-Electrolytic-C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 -> https://www.lcsc.com/product-detail/Through-Hole-Ceramic-Ca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
- C38: value 10 uF -> 0.1uF; LCSC https://www.lcsc.com/product-detail/Aluminum-Electrolytic-C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 -> https://www.lcsc.com/product-detail/Through-Hole-Ceramic-Ca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
- R13, R14, R46, R47, R48, R49, R50, R51, R52, R53, R54, R55, R56, R57, R58, R59, R60, R61, R62, R63, R76: value 10 kO -> 10k
- R15, R16, R17, R18: value 220 O -> 220
- R22, R23, R24, R25: value 4.3 kO -> 4.3k
- R75: value 47 kO -> 47k
- R77: value 47 kO T+-1% -> 47k T+-1%
- R78: value 200 kO -> 200k
- R80: value 120 kO -> 120k
- R81: value 22.1kO -> 22.1k
Connections:
- net Buzzer_Collector: now also Q13.7 (C4), Q13.8 (C4); no longer Q6.7 (C4), Q6.8 (C4)
- net External_LED_Collector_1: now also Q6.7 (C4), Q6.8 (C4); no longer Q13.7 (C4), Q13.8 (C4)
- net External_LED_Collector_3: now also Q16.7 (C4), Q16.8 (C4)
- net GND: now also Q16.10 (E4), Q16.12 (E3), Q16.14 (E2), Q16.16 (E1)
- net Motor_F_Collector_1: now also Q13.3 (C2), Q13.4 (C2); no longer Q6.3 (C2), Q6.4 (C2)
- net Motor_F_Collector_2: now also Q6.3 (C2), Q6.4 (C2); no longer Q13.3 (C2), Q13.4 (C2)
- net Motor_F_Collector_4: now also Q16.3 (C2), Q16.4 (C2)
- net Motor_PWM_Collector_1: now also Q13.1 (C1), Q13.2 (C1); no longer Q6.1 (C1), Q6.2 (C1)
- net Motor_PWM_Collector_2: now also Q6.1 (C1), Q6.2 (C1); no longer Q13.1 (C1), Q13.2 (C1)
- net Motor_PWM_Collector_4: now also Q16.1 (C1), Q16.2 (C1)
- net Motor_R_Collector_1: now also Q13.5 (C3), Q13.6 (C3); no longer Q6.5 (C3), Q6.6 (C3)
- net Motor_R_Collector_2: now also Q6.5 (C3), Q6.6 (C3); no longer Q13.5 (C3), Q13.6 (C3)
- net Motor_R_Collector_4: now also Q16.5 (C3), Q16.6 (C3)
- net STM32 GPIO: now also RN2.5, RN2.6, RN2.7, RN2.8, RN3.5, RN3.6, RN3.7, RN3.8, RN4.5, RN4.6, RN4.7, RN4.8, RN5.5, RN5.6, RN5.7, RN5.8
- net VCC (3V): no longer BZ2.1 (+), D7.1 (K)
- net VCC (5V): now also BZ2.1 (+), D7.1 (K)
- net at Q13.13 (B2): now also RN5.2
- net at Q13.15 (B1): now also RN5.1
- net at Q11.15 (B1): now also RN2.1
- net at Q13.9 (B4): now also RN5.4
- net at Q11.9 (B4): now also RN2.4
- net at Q6.9 (B4): now also RN4.4
- net at Q11.11 (B3): now also RN2.3
- net at Q11.13 (B2): now also RN2.2
- net at Q13.11 (B3): now also RN5.3
- net at Q6.11 (B3): now also RN4.3
- net at Q6.13 (B2): now also RN4.2
- net at Q6.15 (B1): now also RN4.1
- new net: Q16.11 (B3), RN3.3
- new net: Q16.13 (B2), RN3.2
- new net: Q16.15 (B1), RN3.1
- new net: Q16.9 (B4), RN3.4
Other:
- note added: "Consider applying shared connection to this Resistor Array among multiple Encoders or Motor Connectors."
- note added: "TODO: 4. Replace all Through-a-hole/Leaded elements with SMD. 7. Resolve all ERC exceptions and warnings. 9. Recalculate all of the numerical values for scheme, to be sure. 13. Consider implement Multi unit symbols for IC Arrays. 14. Consider applying shared connection to this Resistor Arrays among multiple Encoders or Motor Connectors? 15. Include PWR_FLAG, properly. DONE: 1. Rework transisor sc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"
- note added: "Transistor array (deprecated design)"
- note added: "maybe it needs to be connected to the GND"
- note added: "oh... it's already on the STM32, somehow i forgot these, but maybe this connectors will help us later"
- note removed: "TODO: 4. Replace all Through-a-hole/Leaded elements with SMD. 7. Resolve all ERC exceptions and warnings. 9. Recalculate all of the numerical values for scheme, to be sure. 10. Integrate Resistor/(Capacitors) Networks, Arrays? DONE: 1. Rework transisor schemes with transistor arrays. => DONE 1.1 Motor controllers. => DONE 1.2 External LEDs. => DONE 1.3 Buzzer. => DONE 2. Rework power supply by ta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"
- note removed: "but it can be 5V also"
- moved on the sheet: BZ2, C10, C15, C16, C17, C18, C19, C20, C21, C22, C23, C24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

Commit message: Issue #1: added Ethernet, MPU, reworked LEDs
Parts:
- removed BZ2: Buzzer, symbol Device:Buzzer
- removed C35, C37: 10uF, symbol Device:C
- removed C36, C38: 0.1uF, symbol Device:C
- removed F1, F2, F3, F4: Fuse, symbol Device:Fuse
- removed J22, J23, J24, J3: Encoder, symbol Connector_Generic:Conn_01x04
- removed R56, R57, R58, R59, R60, R61, R62, R63: 10k, symbol Device:R_US
- added BUZZER1: FST-9650B-3V, easyeda2kicad:BUZ-SMD_L9.6-W9.6-LS10.0-R, symbol C391032:FST-9650B-3V
- added BZ3: Buzzer, symbol Device:Buzzer
- added C100, C102, C65, C66, C70, C83, C84, C85, C86, C87, C88, C89, C90, C91, C92, C93, C94, C97, C98: 0.1uF, symbol Device:C
- added C101, C63, C95, C96, C99: 10 uF, symbol Device:C
- added C48, C52, C62, C69: 0.1 uF, symbol Device:C
- added C50, C51, C61: 22 uF, Capacitor_SMD:C_2220_5750Metric, symbol Device:C
- added C64, C67, C68: 10uF, symbol Device:C
- added D12, D13, D14, D15: Blue LED, symbol Device:LED
- added D9: D, symbol Device:D
- added F10, F11, F12, F5, F6, F7, F8, F9: Fuse, symbol Device:Fuse
- added FB1: FerriteBead, symbol Device:FerriteBead
- added J27, J29, J30, J31, J40, J41, J42, J43: Encoder, symbol Connector_Generic:Conn_01x04
- added J36, J37, J38, J39: Motor control, symbol Connector_Generic:Conn_01x04
- added Q14: MMPQ3904, easyeda2kicad:SOIC-16_L9.9-W3.9-P1.27-LS6.0-BL, symbol C904282:MMPQ3904
- added R30, R31, R32, R33, R34, R35, R36, R37, R42, R43, R44, R45: 10k, symbol Device:R_US
- added RN10, RN11, RN12, RN13, RN14: 4D03WGJ0102T5E (10k), easyeda2kicad:RES-ARRAY-SMD_0603-8P-L3.2-W1.6-BL, symbol C20197:4D03WGJ0102T5E
- added U4: KSZ8081RNBIA-TR, easyeda2kicad:QFN-32_L5.0-W5.0-P0.50-BL-EP3.4, symbol C100018:KSZ8081RNBIA-TR
- added U5: MPU-6050_C24112, easyeda2kicad:QFN-24_L4.0-W4.0-P0.50-BL-EP2.7, symbol C24112:MPU-6050_C24112
- C10: value 0.1uF -> 2.2nF; LCSC https://www.lcsc.com/product-detail/Through-Hole-Ceramic-Ca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 -> https://www.lcsc.com/product-detail/Multilayer-Ceramic-Capa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
- C11: value 10uF -> 0.1uF; LCSC https://www.lcsc.com/product-detail/Aluminum-Electrolytic-C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 -> https://www.lcsc.com/product-detail/Multilayer-Ceramic-Capa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
- C15, C17, C20: LCSC https://www.lcsc.com/product-detail/Through-Hole-Ceramic-Ca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 -> https://www.lcsc.com/product-detail/Multilayer-Ceramic-Capa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
- C18, C19: LCSC https://www.lcsc.com/product-detail/Aluminum-Electrolytic-C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 -> https://www.lcsc.com/product-detail/Multilayer-Ceramic-Capa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
- C33: value 10 uF -> 0.1uF; LCSC https://www.lcsc.com/product-detail/Aluminum-Electrolytic-C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 -> https://www.lcsc.com/product-detail/Multilayer-Ceramic-Capa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
- C34: value 0.1 uF -> 10 uF; LCSC https://www.lcsc.com/product-detail/Through-Hole-Ceramic-Ca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 -> https://www.lcsc.com/product-detail/Multilayer-Ceramic-Capa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
- D2, D3, D4, D5: LCSC (none) -> https://www.lcsc.com/product-detail/LED-Indication-Discrete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
- R52, R53, R54, R55: value 10k -> 220; LCSC https://www.lcsc.com/product-detail/Through-Hole-Resistors_TyoHM-RN1-4W10KFT-BA1_C410695.html -> https://www.lcsc.com/product-detail/Through-Hole-Resistors_Huaxing-Mechanical-Elec-MF1-4W-220-1-T52_C714546.html?s_z=n_MF1%2F4W-220R-T52
- RN1: value 4D03WGJ0102T5E (10k) -> 4D03WGJ0102T5E (1k); LCSC https://www.lcsc.com/product-detail/Resistor-Networks-Arrays_UNI-ROYAL-Uniroyal-Elec-4D03WGJ0103T5E_C29718.html?s_z=s_Resistors%257CResistor%2520Networks%252C%2520Arrays -> https://www.lcsc.com/product-detail/Resistor-Networks-Arrays_UNI-ROYAL-Uniroyal-Elec-4D03WGJ0102T5E_C20197.html?s_z=s_Resistors%257CResistor%2520Networks%252C%2520Arrays
Connections:
- net idk, mb some false pin is gone; now on net GND: U6.9 (EP)
- net Buzzer_Collector: now also BUZZER1.2, BZ3.2 (-), D9.2 (A)
- net GND: now also C10.2, C100.1, C101.1, C102.1, C48.1, C50.2, C51.2, C52.1, C61.2, C62.1, C63.1, C64.1, C65.1, C66.1, C67.1, C68.1, C69.1, C70.1, C83.1, C84.1, C85.1, C86.1, C87.1, C88.1, C89.1, C90.1, C91.1, C92.1, C93.1, C94.1, C95.1, C96.1, C97.1, C98.1, C99.1, D12.1 (K), D13.1 (K), D14.1 (K), D15.1 (K), J27.4 (Pin_4), J29.4 (Pin_4), J30.4 (Pin_4), J31.4 (Pin_4), J36.4 (Pin_4), J37.4 (Pin_4), J38.4 (Pin_4), J39.4 (Pin_4), J40.4 (Pin_4), J41.4 (Pin_4), J42.4 (Pin_4), J43.4 (Pin_4), Q14.10 (E4), Q14.12 (E3), Q14.14 (E2), Q14.16 (E1), U4.1 (GND), U5.18 (GND), U5.25 (EP); no longer C10.1, D2.1 (K), D3.1 (K), D4.1 (K), D5.1 (K)
- net Motor_F_Collector_1: now also C24.2, J19.2 (Pin_2), C86.2, J37.2 (Pin_2), R43.1, RN11.4; no longer C23.2, J18.2 (Pin_2), R48.1
- net Motor_F_Collector_2: now also C30.2, J21.2 (Pin_2), R49.1, C92.2, J39.2 (Pin_2), RN12.3; no longer C29.2, J20.2 (Pin_2), R54.1
- net Motor_F_Collector_3: now also C23.2, J18.2 (Pin_2), C85.2, J36.2 (Pin_2), R42.1, RN10.2; no longer C24.2, J19.2 (Pin_2), R49.1
- net Motor_F_Collector_4: now also C29.2, J20.2 (Pin_2), R48.1, C91.2, J38.2 (Pin_2), RN11.1; no longer C30.2, J21.2 (Pin_2), R55.1
- net Motor_PWM_Collector_1: now also C22.2, J19.3 (Pin_3), R14.1, C84.2, J37.3 (Pin_3), RN11.3; no longer C21.2, J18.3 (Pin_3), R46.1
- net Motor_PWM_Collector_2: now also C28.2, J21.3 (Pin_3), R47.1, C90.2, J39.3 (Pin_3), RN12.2; no longer C27.2, J20.3 (Pin_3), R52.1
- net Motor_PWM_Collector_3: now also C21.2, J18.3 (Pin_3), R13.1, C83.2, J36.3 (Pin_3), RN10.1; no longer C22.2, J19.3 (Pin_3), R47.1
- net Motor_PWM_Collector_4: now also C27.2, J20.3 (Pin_3), R46.1, C89.2, J38.3 (Pin_3), RN10.4; no longer C28.2, J21.3 (Pin_3), R53.1
- net Motor_R_Collector_1: now also C26.2, J19.1 (Pin_1), C88.2, J37.1 (Pin_1), R45.1, RN12.1; no longer C25.2, J18.1 (Pin_1), R50.1
- net Motor_R_Collector_2: now also C32.2, J21.1 (Pin_1), R51.1, C94.2, J39.1 (Pin_1), RN12.4; no longer C31.2, J20.1 (Pin_1)
- net Motor_R_Collector_3: now also C25.2, J18.1 (Pin_1), C87.2, J36.1 (Pin_1), R44.1, RN10.3; no longer C26.2, J19.1 (Pin_1), R51.1
- net Motor_R_Collector_4: now also C31.2, J20.1 (Pin_1), R50.1, C93.2, J38.1 (Pin_1), RN11.2; no longer C32.2, J21.1 (Pin_1)
- net VCC (3V): now also R30.2, R31.2, R32.2, R33.2, R34.2, R35.2, R36.2, R37.2, RN13.5, RN13.6, RN13.7, RN13.8, RN14.5, RN14.6, RN14.7, RN14.8; no longer R13.2, R14.2
- net VCC (5V): now also D2.2 (A), D3.2 (A), D4.2 (A), D5.2 (A), R13.2, R14.2, BUZZER1.1 (+), BZ3.1 (+), C100.2, C101.2, C102.2, C63.2, C64.2, C65.2, C66.2, C67.2, C68.2, C69.2, C70.2, C95.2, C96.2, C97.2, C98.2, C99.2, D9.1 (K), F10.2, F11.2, F12.2, F5.2, F6.2, F7.2, F8.2, F9.2, R42.2, R43.2, R44.2, R45.2, RN10.5, RN10.6, RN10.7, RN10.8, RN11.5, RN11.6, RN11.7, RN11.8, RN12.5, RN12.6, RN12.7, RN12.8; no longer C10.2, C11.2, C33.2, C34.2, R52.2, R53.2, R54.2, R55.2
- net LED_Collector_1: now reaches R17.2
- net LED_Collector_1: now also R15.2, R16.2, R18.2, Q14.1 (C1), Q14.2 (C1); no longer D4.2 (A)
- net at RN1.1: now also Q14.15 (B1)
- net at RN1.2: now also Q14.13 (B2)
- net at RN1.3: now also Q14.11 (B3)
- net at RN1.4: now also Q14.9 (B4)
- net Resistor_Array_13: now reaches RN1.5
- net Resistor_Array_13: now also C34.2, J10.1 (Pin_1), J10.2 (Pin_2), J28.1 (Pin_1), J28.2 (Pin_2), J28.3 (Pin_3), J28.4 (Pin_4), J7.1 (Pin_1), J7.2 (Pin_2), J8.1 (Pin_1), J8.2 (Pin_2), R11.1, R19.2, R20.2, R21.2, R26.1, R27.1, R28.1, R29.1, R38.1, R39.1, R40.1, R41.1, R52.1, R53.1, R54.1, R55.1, R7.1, R9.1, RN1.6, RN1.7, RN1.8, RN2.5, RN2.6, RN2.7, RN2.8, RN3.5, RN3.6, RN3.7, RN3.8, RN4.5, RN4.6, RN4.7, RN4.8, RN5.5, RN5.6, RN5.7, RN5.8, J27.1 (Pin_1), J27.2 (Pin_2), J29.1 (Pin_1), J29.2 (Pin_2), J30.1 (Pin_1), J30.2 (Pin_2), J31.1 (Pin_1), J31.2 (Pin_2), J40.1 (Pin_1), J40.2 (Pin_2), J41.1 (Pin_1), J41.2 (Pin_2), J42.1 (Pin_1), J42.2 (Pin_2), J43.1 (Pin_1), J43.2 (Pin_2), R30.1, R31.1, R32.1, R33.1, R34.1, R35.1, R36.1, R37.1, RN13.1, RN13.2, RN13.3, RN13.4, RN14.1, RN14.2, RN14.3, RN14.4, U5.1 (CLKIN), U5.11 (FSYNC), U5.12 (INT), U5.23 (SCL), U5.24 (SDA), U5.7 (AUX_CL), U5.8 (VLOGIC), U5.9 (AD0)
- removed net STM32 GPIO: J10.1 (Pin_1), J10.2 (Pin_2), J28.1 (Pin_1), J28.2 (Pin_2), J28.3 (Pin_3), J28.4 (Pin_4), J7.1 (Pin_1), J7.2 (Pin_2), J8.1 (Pin_1), J8.2 (Pin_2), R11.1, R13.1, R14.1, R15.1, R16.1, R17.1, R18.1, R19.2, R20.2, R21.2, R26.1, R27.1, R28.1, R29.1, R38.1, R39.1, R40.1, R41.1, R7.1, R9.1, RN2.5, RN2.6, RN2.7, RN2.8, RN3.5, RN3.6, RN3.7, RN3.8, RN4.5, RN4.6, RN4.7, RN4.8, RN5.5, RN5.6, RN5.7, RN5.8
- new net: D13.2 (A), R53.2
- new net: C33.2, U5.10 (REGOUT)
- new net: C10.1, U5.20 (CPOUT)
- new net: C61.1, C62.2, U4.2 (VDD_1.2)
- new net: C48.2, C50.1, FB1.2, U4.3 (VDDA_3.3)
- new net: D4.1 (K), R17.1
- new net: F5.1, J27.3 (Pin_3)
- new net: D2.1 (K), R15.1
- new net: D14.2 (A), R54.2
- new net: D12.2 (A), R52.2
- new net: F10.1, J41.3 (Pin_3)
- new net: F7.1, J30.3 (Pin_3)
- new net: D5.1 (K), R18.1
- new net: F8.1, J31.3 (Pin_3)
- new net: D15.2 (A), R55.2
- new net: F9.1, J40.3 (Pin_3)
- new net: F6.1, J29.3 (Pin_3)
- new net: F12.1, J43.3 (Pin_3)
- new net: D3.1 (K), R16.1
- new net: F11.1, J42.3 (Pin_3)
- new net LED_Collector_2: Q14.3 (C2), Q14.4 (C2)
- new net LED_Collector_3: Q14.5 (C3), Q14.6 (C3)
- new net LED_Collector_4: Q14.7 (C4), Q14.8 (C4)
- new net VCC (3.3V): C51.1, C52.2, FB1.1, U4.17 (VDDIO)
- new net VDD (3V): C11.2, U5.13 (VDD)
Other:
- note added: "Encoders (4X) (deprecated design)"
- note added: "Ethernet transreciever"
- note added: "MPU-6050"
- note added: "Motors controllers (4X) (deprecated design)"
- note added: "TODO: 4. Replace all Through-a-hole/Leaded elements with SMD. 4.2 Resister 4.3 Other 7. Resolve all ERC exceptions and warnings. 9. Recalculate all of the numerical values for scheme, to be sure. 13. Consider implement Multi unit symbols for IC Arrays. 15. Include PWR_FLAG, properly. DONE: 1. Rework transisor schemes with transistor arrays. 1.1 Motor controllers. 1.2 External LEDs. 1.3 Buzzer. 2.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"
- note added: "actually, i don't quite understand how to choose suitable ferrite bead. i chose one that is equal to Ethernet frequency and has high impedance. i guess, later, we should replace it with a more suitable. later is when i will properly read the documentation."
- note added: "also, connect paddle to the GND."
- note added: "i guess, idealy resistor should be 117 Ohms. maybe later I will replace it. maybe not."
- note added: "scrapyard"
- note added: "some VLOGIC"
- note added: "the pins will be populated later. when we will know what we need. Andrii is dealing with this."
- note removed: "Consider applying shared connection to this Resistor Array among multiple Encoders or Motor Connectors."
- note removed: "TODO: 4. Replace all Through-a-hole/Leaded elements with SMD. 7. Resolve all ERC exceptions and warnings. 9. Recalculate all of the numerical values for scheme, to be sure. 13. Consider implement Multi unit symbols for IC Arrays. 14. Consider applying shared connection to this Resistor Arrays among multiple Encoders or Motor Connectors? 15. Include PWR_FLAG, properly. DONE: 1. Rework transisor sc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"
- moved on the sheet: BZ1, C1, C12, C13, C14, C15, C16, C17, C18, C19, C2, C20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

Commit message: Issue #1: Replaced resistors, fuses, and diode with SMD ones
Parts:
- removed F10, F11, F12: Fuse, symbol Device:Fuse
- added F1, F2, F3: Fuse, symbol Device:Fuse
- D7: LCSC https://www.lcsc.com/product-detail/Switching-Diodes_LGE-1N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 -> https://www.lcsc.com/product-detail/Schottky-Diodes_JSMSEMI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
- F9: LCSC (none) -> https://www.lcsc.com/product-detail/Resettable-Fuses_BNstar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
- R15, R16, R17, R18, R24, R25: LCSC https://www.lcsc.com/product-detail/Through-Hole-Resistors_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 -> https://www.lcsc.com/product-detail/Chip-Resistor-Surface-M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
Connections:
- net VCC (5V): now also F1.2, F2.2, F3.2
- net at J41.3 (Pin_3): now also F1.1
- net at J43.3 (Pin_3): now also F3.1
- net at J42.3 (Pin_3): now also F2.1
Other:
- note added: "TODO: 7. Resolve all ERC exceptions and warnings. 9. Recalculate all of the numerical values for scheme, to be sure. 13. Consider implement Multi unit symbols for IC Arrays. 15. Include PWR_FLAG, properly. DONE: 1. Rework transisor schemes with transistor arrays. 1.1 Motor controllers. 1.2 External LEDs. 1.3 Buzzer. 2. Rework power supply by taking already in use PMIC in rpi-power-HAT. (Varya PCB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"
- note added: "i'm not sure about this diode."
- note removed: "TODO: 4. Replace all Through-a-hole/Leaded elements with SMD. 4.2 Resister 4.3 Other 7. Resolve all ERC exceptions and warnings. 9. Recalculate all of the numerical values for scheme, to be sure. 13. Consider implement Multi unit symbols for IC Arrays. 15. Include PWR_FLAG, properly. DONE: 1. Rework transisor schemes with transistor arrays. 1.1 Motor controllers. 1.2 External LEDs. 1.3 Buzzer. 2.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"

Commit message: Issue #1: Added XTAL and RJ45 Connector
Parts:
- added C35, C38, C71, C72: 0.1uF, symbol Device:C
- added C36: 22uF, Capacitor_SMD:C_2220_5750Metric, symbol Device:C
- added C37: 2.2uF, Capacitor_SMD:C_2220_5750Metric, symbol Device:C
- added J3: HR911105A_C12074, easyeda2kicad:RJ45-TH_HR911105A, symbol C12074:HR911105A_C12074
- added L3: BLM21PG331SN1D, symbol Device:L
- added R56: 24, symbol Device:R_US
- added R57, R58: 330, symbol Device:R_US
- added X1: X1G004451000400, easyeda2kicad:OSC-SMD_4P-L5.0-W3.2-BL_SG5032, symbol C37076:X1G004451000400
- C48: value 0.1 uF -> 22pF; footprint (none) -> Capacitor_SMD:C_2220_5750Metric; LCSC https://www.lcsc.com/product-detail/Multilayer-Ceramic-Capacitors-MLCC-SMD-SMT_YAGEO-CC0603KRX7R9BB104_C14663.html?s_z=n_100nf%2520smd -> https://www.lcsc.com/product-detail/Multilayer-Ceramic-Capacitors-MLCC-SMD-SMT_YAGEO-CC0603JRNPO9BN220_C105620.html?s_z=n_22%2520pF
- C50: value 22 uF -> 0.1uF; footprint Capacitor_SMD:C_2220_5750Metric -> (none); LCSC C784103 -> https://www.lcsc.com/product-detail/Multilayer-Ceramic-Capa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
- C51, C61: value 22 uF -> 22uF
- C52: value 0.1 uF -> 0.1uF
- C62: value 0.1 uF -> 0.1uF 200V
Connections:
- net GND: now also C50.1, C35.1, C36.2, C37.2, C38.1, C71.2, C72.2, J3.8 (CHSGND), X1.2 (GND); no longer C50.2
- net VCC (3.3V): now also C61.1, L3.1, R57.2, R58.2; no longer C51.1
- net at FB1.2, U4.3 (VDDA_3.3): now also C36.1, C38.2; no longer C48.2, C50.1
- net LED0: now reaches U4.30 (LED0/NWAYEN)
- net LED0: now also J3.10
- net RXM: now reaches U4.4 (RXM)
- net RXM: now also J3.6 (RD-)
- net RXP: now reaches U4.5 (RXP)
- net RXP: now also J3.3 (RD+)
- net TXM: now reaches U4.6 (TXM)
- net TXM: now also J3.2 (TD-)
- net TXP: now reaches U4.7 (TXP)
- net TXP: now also J3.1 (TD+)
- net at U4.9 (XI): now also R56.1
- new net: C62.2, J3.SH1, J3.SH2
- new net: C50.2, C51.1, L3.2, X1.1 (OE/~{ST}), X1.4 (VCC)
- new net: J3.12, R57.1
- new net: C72.1, J3.4
- new net: C48.2, R56.2, X1.3 (OUT)
- new net: C71.1, J3.5
- new net: J3.9, R58.1
- new net: C35.2, C37.1, U4.2 (VDD_1.2)
- no-connect marks 0 -> 2
Other:
- note added: "TODO: 7. Resolve all ERC exceptions and warnings. 9. Recalculate all of the numerical values for scheme, to be sure. 13. Consider implement Multi unit symbols for IC Arrays. 15. Include PWR_FLAG, properly. 22. Add RJ45 Connector's LED STM32 Signal. DONE: 1. Rework transisor schemes with transistor arrays. 1.1 Motor controllers. 1.2 External LEDs. 1.3 Buzzer. 2. Rework power supply by taking alrea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"
- note added: "add lcsc links"
- note added: "here, we can connect OE/ST to the VCC to enable crystal constantly. or control it with XO."
- note added: "signal for led"
- note removed: "TODO: 7. Resolve all ERC exceptions and warnings. 9. Recalculate all of the numerical values for scheme, to be sure. 13. Consider implement Multi unit symbols for IC Arrays. 15. Include PWR_FLAG, properly. DONE: 1. Rework transisor schemes with transistor arrays. 1.1 Motor controllers. 1.2 External LEDs. 1.3 Buzzer. 2. Rework power supply by taking already in use PMIC in rpi-power-HAT. (Varya PCB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"
- moved on the sheet: C15, C19, C20, J11, J8, R24, R25
