File: rover-chasis-controller.kicad_sch (KiCad schematic)
At the start: 266 parts, among them J1 Screw_Terminal_01x02, J10 GPS Interface, J11 Compass Connection (I2C), J12 External LED (Red), J13 External LED (Yellow), J14 External LED (Green), J15 External LED (Red), J16 External LED (Yellow), J17 External LED (Green), J18 Motor control, J19 Motor control, J2 Motor control, J20 Motor control, J21 Motor control, J25 MPU-6050 IMU Module, J26 Screw_Terminal_01x02, J27 Encoder, J28 Conn_01x06, J29 Encoder, J3 HR911105A_C12074, J30 Encoder, J31 Encoder, J36 Motor control, J37 Motor control, J38 Motor control, J39 Motor control, J4 External LED, J40 Encoder, J41 Encoder, J42 Encoder, J43 Encoder, J5 External LED, J6 External LED, J7 TTL, J8 Ultrasonic Sensor Inputs, J9 MPU-6050 IMU Module, Q1 IRF9540N, Q10 MMPQ3904, Q11 MMPQ3904, Q12 SUD50P10-43L-TP, Q13 MMPQ3904, Q14 MMPQ3904, Q15 SUD50P10-43L-TP, Q16 MMPQ3904, Q2 NPN, Q3 NPN, Q4 NPN, Q5 NPN, Q6 MMPQ3904, Q7 NPN, Q8 NPN, Q9 NPN, U1 LD1117S33TR_SOT223, U2 AP64500, U3 TPS5430DDA, U4 KSZ8081RNBIA-TR, U5 MPU-6050_C24112, U6 AP64500SP-13, X1 X1G004451000400

Commit message: Issue #1: Populated pins, small fixes
Parts:
- removed C10: 2.2nF, symbol Device:C
- removed RN13, RN14: 4D03WGJ0102T5E (10k), easyeda2kicad:RES-ARRAY-SMD_0603-8P-L3.2-W1.6-BL, symbol C20197:4D03WGJ0102T5E
- added C73, C76, C77, C80, C81: 0.1uF, symbol Device:C
- added C74, C75, C78, C79: 10 uF, symbol Device:C
- added F10, F11, F12, F4: Fuse, symbol Device:Fuse
- added J22: Ultrasonic Sensor Inputs, symbol Connector_Generic:Conn_01x04
- added J23, J24, J32, J33: Encoder, symbol Connector_Generic:Conn_01x04
- added R59, R60, R61, R62, R63, R71, R72, R73, R74: 24, symbol Device:R_US
- added RN6, RN7: 4D03WGJ0102T5E (10k), easyeda2kicad:RES-ARRAY-SMD_0603-8P-L3.2-W1.6-BL, symbol C20197:4D03WGJ0102T5E
- C34: value 10 uF -> 2.2nF; LCSC https://www.lcsc.com/product-detail/Multilayer-Ceramic-Capacitors-MLCC-SMD-SMT_Samsung-Electro-Mechanics-CL21A106KOQNNNE_C1713.html?s_z=n_10uF%2520smd -> https://www.lcsc.com/product-detail/Multilayer-Ceramic-Capacitors-MLCC-SMD-SMT_YAGEO-CC0402KRX7R9BB222_C106861.html?s_z=n_Ceramic%252C%2520X7R%252C%25202.2nF%2520%25C2%25B110%2525%252C%252050V%2520smd
Connections:
- net ADC: no longer D11.1 (A1), R76.2, R77.1
- net GND: now also C34.2, U5.11 (FSYNC), C73.1, C74.1, C75.1, C76.1, C77.1, C78.1, C79.1, C80.1, C81.1, J22.4 (Pin_4), J23.4 (Pin_4), J24.4 (Pin_4), J32.4 (Pin_4), J33.4 (Pin_4); no longer C34.1
- net Motor_PWM_Collector_1: now also C88.2, J37.1 (Pin_1), RN12.1; no longer C84.2, J37.3 (Pin_3), RN11.3
- net Motor_PWM_Collector_2: now also C94.2, J39.1 (Pin_1), RN12.4; no longer C90.2, J39.3 (Pin_3), RN12.2
- net Motor_PWM_Collector_3: now also C87.2, J36.1 (Pin_1), RN10.3; no longer C83.2, J36.3 (Pin_3), RN10.1
- net Motor_PWM_Collector_4: now also C93.2, J38.1 (Pin_1), RN11.2; no longer C89.2, J38.3 (Pin_3), RN10.4
- net Motor_R_Collector_1: now also C84.2, J37.3 (Pin_3), RN11.3; no longer C88.2, J37.1 (Pin_1), RN12.1
- net Motor_R_Collector_2: now also C90.2, J39.3 (Pin_3), RN12.2; no longer C94.2, J39.1 (Pin_1), RN12.4
- net Motor_R_Collector_3: now also C83.2, J36.3 (Pin_3), RN10.1; no longer C87.2, J36.1 (Pin_1), RN10.3
- net Motor_R_Collector_4: now also C89.2, J38.3 (Pin_3), RN10.4; no longer C93.2, J38.1 (Pin_1), RN11.2
- net STM32 I2C: no longer J11.1 (Pin_1), J11.2 (Pin_2), R24.2, R25.2
- net VCC (3V): now also RN6.5, RN6.6, RN6.7, RN6.8, RN7.5, RN7.6, RN7.7, RN7.8
- net VCC (5V): now also C73.2, C74.2, C75.2, C76.2, C77.2, C78.2, C79.2, C80.2, C81.2, F10.2, F11.2, F12.2, F4.2, J22.3 (Pin_3)
- net VDD (3V): now also C33.2; no longer C11.2
- net at U5.10 (REGOUT): now also C11.2; no longer C33.2
- net at U5.20 (CPOUT): now also C34.1
- net STM32 GPIO: now reaches J3.11
- net STM32 GPIO: now also J27.1 (Pin_1), J27.2 (Pin_2), J28.1 (Pin_1), J28.2 (Pin_2), J28.3 (Pin_3), J28.4 (Pin_4), J29.1 (Pin_1), J29.2 (Pin_2), J30.1 (Pin_1), J30.2 (Pin_2), J31.1 (Pin_1), J31.2 (Pin_2), R11.1, R19.2, R20.2, R21.2, R26.1, R27.1, R28.1, R29.1, R30.1, R31.1, R32.1, R33.1, R34.1, R35.1, R36.1, R37.1, R38.1, R39.1, R40.1, R41.1, R52.1, R53.1, R54.1, R55.1, R7.1, R9.1
- net MDIO: now reaches U4.11 (MDIO)
- net MDIO: now also R61.2
- net MDC: now reaches U4.12 (MDC)
- net MDC: now also R59.2
- net RXD1: now reaches U4.15 (RXD1/PHYAD2)
- net RXD1: now also R74.2
- net RXD0: now reaches U4.16 (RXD0/DUPLEX)
- net RXD0: now also R73.2
- net CRS_DV: now reaches U4.18 (CRS_DV/CONFIG2)
- net CRS_DV: now also R62.2
- net REF_CLK: now reaches U4.19 (REF_CLK/B-CAST_OFF)
- net REF_CLK: now also R60.2
- net TX_EN: now reaches U4.23 (TXEN)
- net TX_EN: now also R63.2
- net TXD0: now reaches U4.24 (TXD0)
- net TXD0: now also R71.2
- net TXD1: now reaches U4.25 (TXD1)
- net TXD1: now also R72.2
- net ETH_REF_CLK: now reaches TB1.P1_11 (PA1)
- net ETH_REF_CLK: now also R60.1
- net TTL_TX: now reaches TB1.P1_12 (PA0-WKUP)
- net TTL_TX: now also J7.2 (Pin_2)
- net MOTOR2_PWM: now reaches TB1.P1_13 (PA3)
- net MOTOR2_PWM: now also RN4.8
- net ETH_MDIO: now reaches TB1.P1_14 (PA2)
- net ETH_MDIO: now also R61.1
- net ENC2_A: now reaches TB1.P1_15 (PA5)
- net ENC2_A: now also J41.1 (Pin_1), J32.1 (Pin_1), RN6.3
- net POWER_SUPPLY_ADC: now reaches TB1.P1_16 (PA4)
- net POWER_SUPPLY_ADC: now also D11.1 (A1), R76.2, R77.1
- net ETH_CRS_DV: now reaches TB1.P1_17 (PA7)
- net ETH_CRS_DV: now also R62.1
- net ENC3_A: now reaches TB1.P1_18 (PA6)
- net ENC3_A: now also J43.1 (Pin_1), J24.1 (Pin_1), RN7.1
- net ETH_RXD1: now reaches TB1.P1_19 (PC5)
- net ETH_RXD1: now also R74.1
- net ETH_RXD0: now reaches TB1.P1_20 (PC4)
- net ETH_RXD0: now also R73.1
- net MOTOR4_PWM: now reaches TB1.P1_21 (PB1)
- net MOTOR4_PWM: now also RN3.8
- net MOTOR3_PWM: now reaches TB1.P1_22 (PB0)
- net MOTOR3_PWM: now also RN2.8
- net BUZZER_OUT: now reaches TB1.P1_24 (PB2)
- net BUZZER_OUT: now also RN5.5
- net LED_YELLOW: now reaches TB1.P1_25 (PE7)
- net LED_YELLOW: now also RN2.5
- net LED_GREEN: now reaches TB1.P1_26 (PE8)
- net LED_GREEN: now also RN3.5
- net ENC1_A: now reaches TB1.P1_27 (PE9)
- net ENC1_A: now also J40.1 (Pin_1), J23.1 (Pin_1), RN6.1
- net ENC1_B: now reaches TB1.P1_29 (PE11)
- net ENC1_B: now also J40.2 (Pin_2), J23.2 (Pin_2), RN6.2
- net US_SENSOR1_ECHO: now reaches TB1.P1_31 (PE13)
- net US_SENSOR1_ECHO: now also J8.2 (Pin_2)
- net US_SENSOR2_ECHO: now reaches TB1.P1_32 (PE14)
- net US_SENSOR2_ECHO: now also J22.2 (Pin_2)
- net MOTOR1_PWM: now reaches TB1.P1_34 (PB10)
- net MOTOR1_PWM: now also RN5.8
- net ETH_TX_EN: now reaches TB1.P1_35 (PB11)
- net ETH_TX_EN: now also R63.1
- net ETH_TXD0: now reaches TB1.P1_36 (PB12)
- net ETH_TXD0: now also R71.1
- net ETH_TXD1: now reaches TB1.P1_37 (PB13)
- net ETH_TXD1: now also R72.1
- net MOTOR3_FWD: now reaches TB1.P1_38 (PB14)
- net MOTOR3_FWD: now also RN2.7
- net MOTOR4_FWD: now reaches TB1.P1_39 (PB15)
- net MOTOR4_FWD: now also RN3.7
- net MOTOR1_FWD: now reaches TB1.P1_40 (PD8)
- net MOTOR1_FWD: now also RN5.7
- net MOTOR2_FWD: now reaches TB1.P1_41 (PD9)
- net MOTOR2_FWD: now also RN4.7
- net US_SENSOR1_TRIG: now reaches TB1.P1_42 (PD10)
- net US_SENSOR1_TRIG: now also J8.1 (Pin_1)
- net US_SENSOR2_TRIG: now reaches TB1.P1_43 (PD11)
- net US_SENSOR2_TRIG: now also J22.1 (Pin_1)
- net ENC4_A: now reaches TB1.P1_44 (PD12)
- net ENC4_A: now also J42.1 (Pin_1), J33.1 (Pin_1), RN7.3
- net ENC4_B: now reaches TB1.P1_45 (PD13)
- net ENC4_B: now also J42.2 (Pin_2), J33.2 (Pin_2), RN7.4
- net ETH_MDC: now reaches TB1.P1_7 (PC1)
- net ETH_MDC: now also R59.1
- net LED_RED: now reaches TB1.P2_11 (PE6)
- net LED_RED: now also RN4.5
- net LED_BLUE_3: now reaches TB1.P2_13 (PE4)
- net LED_BLUE_3: now also RN1.6
- net LED_BLUE_4: now reaches TB1.P2_14 (PE5)
- net LED_BLUE_4: now also RN1.5
- net LED_BLUE_1: now reaches TB1.P2_15 (PE2)
- net LED_BLUE_1: now also RN1.8
- net LED_BLUE_2: now reaches TB1.P2_16 (PE3)
- net LED_BLUE_2: now also RN1.7
- net COMPASS_SCL: now reaches TB1.P2_23 (PB6)
- net COMPASS_SCL: now also J11.2 (Pin_2), R25.2
- net COMPASS_SDA: now reaches TB1.P2_24 (PB7)
- net COMPASS_SDA: now also J11.1 (Pin_1), R24.2
- net ENC2_B: now reaches TB1.P2_28 (PB3)
- net ENC2_B: now also J41.2 (Pin_2), J32.2 (Pin_2), RN6.4
- net MOTOR3_RVR: now reaches TB1.P2_29 (PD5)
- net MOTOR3_RVR: now also RN2.6
- net MOTOR4_RVR: now reaches TB1.P2_30 (PD6)
- net MOTOR4_RVR: now also RN3.6
- net MOTOR1_RVR: now reaches TB1.P2_31 (PD3)
- net MOTOR1_RVR: now also RN5.6
- net MOTOR2_RVR: now reaches TB1.P2_32 (PD4)
- net MOTOR2_RVR: now also RN4.6
- net GPS_RX: now reaches TB1.P2_34 (PD2)
- net GPS_RX: now also J10.1 (Pin_1)
- net GPS_TX: now reaches TB1.P2_35 (PC12)
- net GPS_TX: now also J10.2 (Pin_2)
- net TTL_RX: now reaches TB1.P2_38 (PC11)
- net TTL_RX: now also J7.1 (Pin_1)
- net MPU_SCL: now reaches TB1.P2_43 (PA8)
- net MPU_SCL: now also U5.23 (SCL)
- net MPU_SDA: now reaches TB1.P2_46 (PC9)
- net MPU_SDA: now also U5.24 (SDA)
- net ENC3_B: now reaches TB1.P2_48 (PC7)
- net ENC3_B: now also J43.2 (Pin_2), J24.2 (Pin_2), RN7.2
- removed net Resistor_Array_13: C34.2, J10.1 (Pin_1), J10.2 (Pin_2), J27.1 (Pin_1), J27.2 (Pin_2), J28.1 (Pin_1), J28.2 (Pin_2), J28.3 (Pin_3), J28.4 (Pin_4), J29.1 (Pin_1), J29.2 (Pin_2), J30.1 (Pin_1), J30.2 (Pin_2), J31.1 (Pin_1), J31.2 (Pin_2), J40.1 (Pin_1), J40.2 (Pin_2), J41.1 (Pin_1), J41.2 (Pin_2), J42.1 (Pin_1), J42.2 (Pin_2), J43.1 (Pin_1), J43.2 (Pin_2), J7.1 (Pin_1), J7.2 (Pin_2), J8.1 (Pin_1), J8.2 (Pin_2), R11.1, R19.2, R20.2, R21.2, R26.1, R27.1, R28.1, R29.1, R30.1, R31.1, R32.1, R33.1, R34.1, R35.1, R36.1, R37.1, R38.1, R39.1, R40.1, R41.1, R52.1, R53.1, R54.1, R55.1, R7.1, R9.1, RN1.5, RN1.6, RN1.7, RN1.8, RN2.5, RN2.6, RN2.7, RN2.8, RN3.5, RN3.6, RN3.7, RN3.8, RN4.5, RN4.6, RN4.7, RN4.8, RN5.5, RN5.6, RN5.7, RN5.8, U5.1 (CLKIN), U5.11 (FSYNC), U5.12 (INT), U5.23 (SCL), U5.24 (SDA), U5.7 (AUX_CL), U5.8 (VLOGIC), U5.9 (AD0)
- new net: F10.1, J24.3 (Pin_3)
- new net: F12.1, J33.3 (Pin_3)
- new net: F11.1, J32.3 (Pin_3)
- new net: F4.1, J23.3 (Pin_3)
Other:
- note added: "Compass Connector"
- note added: "If enccoders are open-drain."
- note added: "SCL"
- note added: "TODO: 7. Resolve all ERC exceptions and warnings. 9. Recalculate all of the numerical values for scheme, to be sure. 13. Consider implement Multi unit symbols for IC Arrays. 15. Include PWR_FLAG, properly. DONE: 1. Rework transisor schemes with transistor arrays. 1.1 Motor controllers. 1.2 External LEDs. 1.3 Buzzer. 2. Rework power supply by taking already in use PMIC in rpi-power-HAT. (Varya PCB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"
- note added: "Ultrasonic Sensor (1)"
- note added: "Ultrasonic Sensor (2)"
- note added: "special pin in open-drain mode."
- note added: "Коли використовувати VLOGIC: Якщо ви підключаєте MPU-6050 до мікроконтролера, який працює на логічних рівнях 1.8В або 5В, тоді ви можете використовувати VLOGIC для встановлення рівнів логіки, сумісних із мікроконтролером. VLOGIC дозволяє забезпечити сумісність між рівнями сигналів I2C (SDA/SCL) і рівнями GPIO мікроконтролера. Коли можна обійтися без VLOGIC: Якщо ваш STM32 працює на 3.3В, як і сам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"
- note added: "це ось достатнє базове підключення"
- note removed: "Compas Connector"
- note removed: "TODO: 7. Resolve all ERC exceptions and warnings. 9. Recalculate all of the numerical values for scheme, to be sure. 13. Consider implement Multi unit symbols for IC Arrays. 15. Include PWR_FLAG, properly. 22. Add RJ45 Connector's LED STM32 Signal. DONE: 1. Rework transisor schemes with transistor arrays. 1.1 Motor controllers. 1.2 External LEDs. 1.3 Buzzer. 2. Rework power supply by taking alrea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"
- note removed: "Ultrasonic Sensor Inputs"
- note removed: "signal for led"
- note removed: "some VLOGIC"
- moved on the sheet: C100, C101, C102, C15, C17, C18, C19, C20, C35, C36, C37, C38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

Commit message: Issue #1: Sketched a rough preliminary PCB design layout
Parts:
- removed BUZZER1: FST-9650B-3V, easyeda2kicad:BUZ-SMD_L9.6-W9.6-LS10.0-R, symbol C391032:FST-9650B-3V
- removed BZ1, BZ3: Buzzer, symbol Device:Buzzer
- removed C12, C13, C14, C47, C69: 0.1 uF, symbol Device:C
- removed C16, C21, C22, C23, C24, C25, C26, C27, C28, C29, C30, C31, C32, C35, C38, C49, C50, C52, C65, C66, C70, C76, C77, C80, C81: 0.1uF, symbol Device:C
- removed C36, C51, C61: 22uF, Capacitor_SMD:C_2220_5750Metric, symbol Device:C
- removed C37: 2.2uF, Capacitor_SMD:C_2220_5750Metric, symbol Device:C
- removed C39: 10uF, Capacitor_SMD:C_2220_5750Metric, symbol Device:C
- removed C4: 220 µF, symbol Device:C_Polarized_US
- removed C40: 2.7nF, Capacitor_SMD:C_0805_2012Metric, symbol Device:C
- removed C41: 100nF, Capacitor_SMD:C_0805_2012Metric, symbol Device:C
- removed C42: 39pF, Capacitor_SMD:C_0805_2012Metric, symbol Device:C
- removed C43: 47pF, Capacitor_SMD:C_0805_2012Metric, symbol Device:C
- removed C44, C45, C46: 22 uF, Capacitor_SMD:C_2220_5750Metric, symbol Device:C
- removed C48: 22pF, Capacitor_SMD:C_2220_5750Metric, symbol Device:C
- removed C5: 10 uF, symbol Device:C_Polarized
- removed C6: 22 uF, symbol Device:C_Polarized
- removed C63, C74, C75, C78, C79: 10 uF, symbol Device:C
- removed C64, C67, C68: 10uF, symbol Device:C
- removed D1: B340A, symbol Device:D_Schottky
- removed D12, D13, D14, D15, D2, D3, D4, D5: Blue LED, symbol Device:LED
- removed D6, D9: D, symbol Device:D
- removed D8: SMF5V0A, Diode_SMD:D_SMF, symbol Diode:SMF5V0A
- removed F10, F11, F12, F4, F5, F6, F7, F8: Fuse, symbol Device:Fuse
- removed J1: Screw_Terminal_01x02, symbol Connector:Screw_Terminal_01x02
- removed J12: External LED (Red), symbol Connector_Generic:Conn_01x02
- removed J13: External LED (Yellow), symbol Connector_Generic:Conn_01x02
- removed J14: External LED (Green), symbol Connector_Generic:Conn_01x02
- removed J18, J19, J2, J20, J21: Motor control, symbol Connector_Generic:Conn_01x04
- removed J23, J24, J27, J29, J30, J31, J32, J33: Encoder, symbol Connector_Generic:Conn_01x04
- removed J25, J9: MPU-6050 IMU Module, symbol Connector_Generic:Conn_01x04
- removed J28: Conn_01x06, symbol Connector_Generic:Conn_01x06
- removed J4, J5, J6: External LED, symbol Connector_Generic:Conn_01x03
- removed L1: 22 µH, symbol Device:L_Iron
- removed L2: 4.7uH, YSPI0724-4R7M:IND-SMD_L7.3-W6.6_YSPI07XX, symbol Device:L
- removed L3: BLM21PG331SN1D, symbol Device:L
- removed Q1: IRF9540N, Package_TO_SOT_THT:TO-220-3_Vertical, symbol Transistor_FET:IRF9540N
- removed Q10, Q11, Q13, Q14, Q16, Q6: MMPQ3904, easyeda2kicad:SOIC-16_L9.9-W3.9-P1.27-LS6.0-BL, symbol C904282:MMPQ3904
- removed Q12: SUD50P10-43L-TP, Package_TO_SOT_SMD:TO-252-2, symbol Transistor_FET:SUD50P10-43L
- removed Q2, Q3, Q4, Q5, Q7, Q8, Q9: NPN, symbol Simulation_SPICE:NPN
- removed R10, R12, R3, R4, R5, R8: 10 kO, symbol Device:R_US
- removed R11, R26, R27, R28, R29, R38, R39, R40, R41, R7, R9: 1 kO, symbol Device:R_US
- removed R13, R14, R30, R31, R32, R33, R34, R35, R36, R37, R42, R43, R44, R45, R46, R47, R48, R49, R50, R51: 10k, symbol Device:R_US
- removed R19, R20, R21: 330 O, symbol Device:R_US
- removed R2: 3.24 kO, symbol Device:R_US
- removed R22, R23: 4.3k, symbol Device:R_US
- removed R52, R53, R54, R55: 220, symbol Device:R_US
- removed R56: 24, symbol Device:R_US
- removed R6: 47 kO T+-1%, symbol Device:R_US
- removed R64: 47k, Resistor_SMD:R_0805_2012Metric, symbol Device:R
- removed R65: 200k, Resistor_SMD:R_0805_2012Metric, symbol Device:R
- removed R66: 16k, Resistor_SMD:R_0805_2012Metric, symbol Device:R
- removed R67: 120k, Resistor_SMD:R_0805_2012Metric, symbol Device:R
- removed R68: 22.1k, Resistor_SMD:R_0805_2012Metric, symbol Device:R
- removed R69, R70: 4.3 kO, symbol Device:R_US
- removed RN6, RN7: 4D03WGJ0102T5E (10k), easyeda2kicad:RES-ARRAY-SMD_0603-8P-L3.2-W1.6-BL, symbol C20197:4D03WGJ0102T5E
- removed TP1: TestPoint, symbol Connector:TestPoint
- removed U1: LD1117S33TR_SOT223, Package_TO_SOT_SMD:SOT-223-3_TabPin2, symbol Regulator_Linear:LD1117S33TR_SOT223
- removed U2: AP64500, ultralibAP64500:AP64500SP-13, symbol dcdc-lib:AP64500
- removed U3: TPS5430DDA, Package_SO:TI_SO-PowerPAD-8_ThermalVias, symbol Regulator_Switching:TPS5430DDA
- removed U4: KSZ8081RNBIA-TR, easyeda2kicad:QFN-32_L5.0-W5.0-P0.50-BL-EP3.4, symbol C100018:KSZ8081RNBIA-TR
- added BUZZER2: YS-SBZ9650DYB05_C409830, easyeda2kicad:BUZ-SMD_L9.6-W9.6-LS10.0-R, symbol C409830:YS-SBZ9650DYB05_C409830
- added C4, C6: 0.1uF, Capacitor_SMD:C_0603_1608Metric, symbol Device:C
- added C5: 22pF, Capacitor_SMD:C_2220_5750Metric, symbol Device:C
- added L1: BLM21PG331SN1D, Inductor_SMD:L_0805_2012Metric, symbol Device:L
- added U1, U2, U3, U7: APT2012LVBC/D, easyeda2kicad:LED-SMD_L2.0-W1.3-R-RD, symbol C5879383:APT2012LVBC_D
- added U4: KSZ8081RNAIA-TR, easyeda2kicad:QFN-24_L4.0-W4.0-P0.50-BL-EP2.6, symbol C145623:KSZ8081RNAIA-TR
- C1: value 4.7 uF -> 0.1uF; footprint (none) -> Capacitor_SMD:C_0603_1608Metric; LCSC https://www.lcsc.com/product-detail/Multilayer-Ceramic-Capacitors-MLCC-SMD-SMT_Murata-Electronics-GRM1885C1H103JA01D_C85973.html?s_z=n_Murata%20GRM1885C1H103JA01D -> https://www.lcsc.com/product-detail/Multilayer-Ceramic-Capacitors-MLCC-SMD-SMT_YAGEO-CC0603KRX7R9BB104_C14663.html?s_z=n_100nf%2520smd; LCSC Part (none) -> C14663
- C100, C102, C11, C15, C17, C20, C33, C62, C71, C72, C73, C83, C84, C85, C86, C87, C88, C89, C90, C91, C92, C93, C94, C97, C98: footprint (none) -> Capacitor_SMD:C_0603_1608Metric; LCSC Part (none) -> C14663
- C101, C18, C19, C95, C96, C99: footprint (none) -> Capacitor_SMD:C_0805_2012Metric; LCSC Part (none) -> C1713
- C2: value 4.7 uF -> 22uF; footprint (none) -> Capacitor_SMD:C_2220_5750Metric; LCSC https://www.lcsc.com/product-detail/Multilayer-Ceramic-Capa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 -> C784103; LCSC Part (none) -> C784103
- C3: value 0.01 uF -> 2.2uF; footprint (none) -> Capacitor_SMD:C_2220_5750Metric; LCSC https://www.lcsc.com/product-detail/Multilayer-Ceramic-Capacitors-MLCC-SMD-SMT_YAGEO-CC0603KRX7R9BB104_C14663.html -> https://www.lcsc.com/product-detail/Multilayer-Ceramic-Capacitors-MLCC-SMD-SMT_Samsung-Electro-Mechanics-CL10A225KO8NNNC_C23630.html?s_z=n_2.2%25CE%25BCF; LCSC Part (none) -> C23630
- C34: footprint (none) -> Capacitor_SMD:C_01005_0402Metric; LCSC Part (none) -> C106861
- C53: LCSC Part (none) -> C13585
- C54: LCSC Part (none) -> C28233
- C55: LCSC Part (none) -> C5375904
- C56: LCSC Part (none) -> C107117
- C57: LCSC Part (none) -> C113821
- C58, C59, C60: LCSC Part (none) -> C784103
- C7, C9: value 0.1 uF -> 22uF; footprint (none) -> Capacitor_SMD:C_2220_5750Metric; LCSC https://www.lcsc.com/product-detail/Through-Hole-Ceramic-Ca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 -> C784103; LCSC Part (none) -> C784103
- C8: value 0.1 uF -> 0.1uF; footprint (none) -> Capacitor_SMD:C_0603_1608Metric; LCSC https://www.lcsc.com/product-detail/Through-Hole-Ceramic-Ca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 -> https://www.lcsc.com/product-detail/Multilayer-Ceramic-Capa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; LCSC Part (none) -> C14663
- D10: LCSC Part (none) -> C42387343
- D11: LCSC Part (none) -> C113952
- D7: footprint (none) -> Diode_SMD:D_SOD-323; LCSC Part (none) -> C2927280
- F1, F2, F3, F9: footprint (none) -> Fuse:Fuse_1812_4532Metric; LCSC Part (none) -> C2760284
- FB1: footprint (none) -> Inductor_SMD:L_0603_1608Metric; LCSC Part (none) -> C160981
- J10, J11, J22, J36, J37, J38, J39, J40, J41, J42, J43, J8: footprint (none) -> Connector_JST:JST_PH_B4B-PH-K_1x04_P2.00mm_Vertical; LCSC Part (none) -> C111514
- J15, J16, J17: footprint (none) -> Connector_JST:JST_PH_B2B-PH-K_1x02_P2.00mm_Vertical; LCSC Part (none) -> C495693
- J26: footprint (none) -> TerminalBlock:TerminalBlock_Altech_AK300-2_P5.00mm; LCSC Part (none) -> C474881
- J7: footprint (none) -> Connector_JST:JST_PH_B3B-PH-K_1x03_P2.00mm_Vertical; LCSC Part (none) -> C265393
- L4: footprint YSPI0724-4R7M:IND-SMD_L7.3-W6.6_YSPI07XX -> easyeda2kicad:IND-SMD_L7.0-W6.6; LCSC C22463813 -> (none); LCSC Part (none) -> C524606
- Q15: LCSC Part (none) -> C41408089
- R1: value 10 kO -> 24; footprint (none) -> Resistor_SMD:R_2512_6332Metric; LCSC https://www.lcsc.com/product-detail/Through-Hole-Resistors_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 -> https://www.lcsc.com/product-detail/Chip-Resistor-Surface-M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; LCSC Part (none) -> C2999627
- R15, R16, R17, R18: footprint (none) -> Resistor_SMD:R_2512_6332Metric; LCSC Part (none) -> C2930459
- R24, R25: footprint (none) -> Resistor_SMD:R_1210_3225Metric; LCSC Part (none) -> C3000632
- R57, R58: footprint (none) -> Resistor_SMD:R_0201_0603Metric; LCSC Part (none) -> C23138
- R59, R60, R61, R62, R63: footprint (none) -> Resistor_SMD:R_2512_6332Metric; LCSC Part (none) -> C2934100
- R71, R72, R73, R74: footprint (none) -> Resistor_SMD:R_2512_6332Metric; LCSC Part (none) -> C2907018
- R75: footprint (none) -> Resistor_SMD:R_0201_0603Metric; LCSC Part (none) -> C98220
- R76: footprint (none) -> Resistor_SMD:R_1206_3216Metric; LCSC https://www.lcsc.com/product-detail/Through-Hole-Resistors_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 -> (none); LCSC Part (none) -> C17902
- R77: footprint (none) -> Resistor_SMD:R_1206_3216Metric; LCSC https://www.lcsc.com/product-detail/Through-Hole-Resistors_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 -> (none); LCSC Part (none) -> C25833
- R78: footprint (none) -> Resistor_SMD:R_0805_2012Metric; LCSC Part (none) -> C728645
- R79: value 16 kO -> 16k; footprint (none) -> Resistor_SMD:R_0805_2012Metric; LCSC Part (none) -> C865809
- R80: footprint (none) -> Resistor_SMD:R_0805_2012Metric; LCSC Part (none) -> C865161
- R81: footprint (none) -> Resistor_SMD:R_0805_2012Metric; LCSC Part (none) -> C2692772
- TB1: LCSC Part (none) -> C118360
- U5: footprint easyeda2kicad:QFN-24_L4.0-W4.0-P0.50-BL-EP2.7 -> easyeda2kicad:QFN-24_L4.0-W4.0-P0.50-BL-EP2.6
- U6: footprint easyeda2kicad:SO-8_L4.9-W3.9-P1.27-LS6.0-BL-EP -> easyeda2kicad:SOIC-8_L4.9-W3.9-P1.27-LS6.0-BL-EP-1; LCSC Part C2070920 -> C2071517
Connections:
- net Buzzer_Collector: now also BUZZER2.2 (-)
- net CRS_DV: now also U4.15 (CRS_DV/PHYAD[1:0])
- net GND: now also C2.2, C3.2, C9.2, C4.1, C5.1, C6.1, U4.22 (GND); no longer C2.1, C9.1
- net LED0: now also U4.23 (LED0/ANEN_SPEED)
- net MDC: now also U4.11 (MDC)
- net MDIO: now also U4.10 (MDIO)
- net REF_CLK: now also U4.16 (REF_CLK)
- net RXD0: now also U4.13 (RXD0)
- net RXD1: now also U4.12 (RXD1)
- net RXM: now also U4.3 (RXM)
- net RXP: now also U4.4 (RXP)
- net TXD0: now also U4.20 (TXD0)
- net TXD1: now also U4.21 (TXD1)
- net TXM: now also U4.5 (TXM)
- net TXP: now also U4.6 (TXP)
- net TX_EN: now also U4.19 (TXEN)
- net VCC (3.3V): now also C8.2, C9.1, L1.1, U4.14 (VDDIO)
- net VCC (5V): now also BUZZER2.1 (+), U1.1 (A), U2.1 (A), U3.1 (A), U7.1 (A)
- net at X1.1 (OE/~{ST}), X1.4 (VCC): now also C7.1, C6.2, L1.2
- net at C1.2: now also C3.1, U4.1 (VDD_1.2); no longer C2.2
- net transistor_array/B3: now reaches RN3.3
- net transistor_array/B2: now reaches RN3.2
- net transistor_array/B1: now reaches RN3.1
- net transistor_array/B4: now reaches RN3.4
- net at R18.1: now also U7.2 (K)
- net at FB1.2: now also C2.1, C4.2, U4.2 (VDDA_3.3)
- net at R17.1: now also U3.2 (K)
- net at R1.2: now also X1.3 (OUT), C5.2
- net transistor_array2/B1: now reaches RN4.1
- net transistor_array2/B2: now reaches RN4.2
- net transistor_array2/B3: now reaches RN4.3
- net transistor_array2/B4: now reaches RN4.4
- net at R15.1: now also U1.2 (K)
- net transistor_array1/B3: now reaches RN2.3
- net transistor_array1/B2: now reaches RN2.2
- net transistor_array1/B1: now reaches RN2.1
- net transistor_array1/B4: now reaches RN2.4
- net transistor_array3/B3: now reaches RN5.3
- net transistor_array3/B2: now reaches RN5.2
- net transistor_array3/B1: now reaches RN5.1
- net transistor_array3/B4: now reaches RN5.4
- net at R16.1: now also U2.2 (K)
- net transistor_array4/B1: now reaches RN1.1
- net transistor_array4/B2: now reaches RN1.2
- net transistor_array4/B3: now reaches RN1.3
- net transistor_array4/B4: now reaches RN1.4
- net VCC: no longer names the net of R1.1
- net VCC: now also U4.8 (XI); no longer C3.1
Other:
- added sheet transistor_array (transistor_array.kicad_sch)
- added sheet transistor_array1 (transistor_array.kicad_sch)
- added sheet transistor_array2 (transistor_array.kicad_sch)
- added sheet transistor_array3 (transistor_array.kicad_sch)
- added sheet transistor_array4 (transistor_array.kicad_sch)
- note removed: "4X"
- note removed: "Add Supressor"
- note removed: "Buzzer (deprecated design)"
- note removed: "CS"
- note removed: "Encoders (4X) (deprecated design)"
- note removed: "External LEDs (deprecated design)"
- note removed: "I calculated value of R4, C4, R3 using formula in AP64500 doc."
- note removed: "If enccoders are open-drain."
- note removed: "Input voltage regulator"
- note removed: "LD111... is adjustable PMIC, need to rework scheme"
- note removed: "LED"
- note removed: "LIS3DSH (I2C) (Accelerometer STM32)"
- note removed: "LIS3DSH (SPI) (Accelerometer STM32)"
- note removed: "MISO"
- note removed: "MOSI"
- note removed: "MPU-6050 IMU Module (deprecated design)"
- note removed: "Motion sensor (STM32F4 user manual) The ST-MEMS motion sensor is an ultra-compact low-power three-axis linear accelerometer. The motion sensor includes a sensing element and an IC interface able to provide the measured acceleration to the external world through the I2C/SPI serial interfaces. The STM32F407VG microcontroller controls this motion sensor through the SPI interface"
- note removed: "Motor controller (deprecated design)"
- note removed: "Motors controllers (4X) (deprecated design)"
- note removed: "Power Supply (deprecated design)"
- note removed: "SCK"
- note removed: "SDL"
- note removed: "Transistor array (deprecated design)"
- note removed: "Two options of LIS3DSH connection."
- note removed: "VCC(3.3V)"
- note removed: "maybe interrupt pins: INT1/DRDY, INT2 (if we want to use interrupts)."
- note removed: "maybe rework this to be a module, not connector and maybe there is one accelerometer on the STM32"
- note removed: "maybe there is already 5V to 3V PMIC in STM32"
- note removed: "maybe, bypass capacitors for noise reducing"
- note removed: "oh... it's already on the STM32, somehow i forgot these, but maybe this connectors will help us later"
- note removed: "scrapyard"
- note removed: "to rework with a PMIC from PowerHat-blablabla... (PCB of Varya)"
- note removed: "to rework with transistor arrays"
- note removed: "voltage divider for the voltage measurment with STM's ADC, but i am not sure about this implementation"
- moved on the sheet: C100, C101, C102, C11, C33, C34, C53, C54, C55, C56, C57, C58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

Commit message: Issue #1: Revised possible PCB design
Parts:
- removed C17, C71, C72, C83, C84, C85, C86, C87, C88, C89, C90, C91, C92, C93, C94: 0.1uF, Capacitor_SMD:C_0603_1608Metric, symbol Device:C
- removed C18: 10uF, Capacitor_SMD:C_0805_2012Metric, symbol Device:C
- removed C53: 10uF, Capacitor_SMD:C_2220_5750Metric, symbol Device:C
- removed C54: 100nF, Capacitor_SMD:C_0805_2012Metric, symbol Device:C
- removed C55: 2.7nF, Capacitor_SMD:C_0805_2012Metric, symbol Device:C
- removed C56: 39pF, Capacitor_SMD:C_0805_2012Metric, symbol Device:C
- removed C57: 47pF, Capacitor_SMD:C_0805_2012Metric, symbol Device:C
- removed C58, C59, C60: 22 uF, Capacitor_SMD:C_2220_5750Metric, symbol Device:C
- removed C62: 0.1uF 200V, Capacitor_SMD:C_0603_1608Metric, symbol Device:C
- removed D10: SMF5V0A, Diode_SMD:D_SMF, symbol Diode:SMF5V0A
- removed D11: SMAJ5.0A, Diode_SMD:D_SMA, symbol Diode:SMAJ5.0A
- removed FB1: FerriteBead, Inductor_SMD:L_0603_1608Metric, symbol Device:FerriteBead
- removed J10: GPS Interface, Connector_JST:JST_PH_B4B-PH-K_1x04_P2.00mm_Vertical, symbol Connector_Generic:Conn_01x04
- removed J26: Screw_Terminal_01x02, TerminalBlock:TerminalBlock_Altech_AK300-2_P5.00mm, symbol Connector:Screw_Terminal_01x02
- removed J3: HR911105A_C12074, easyeda2kicad:RJ45-TH_HR911105A, symbol C12074:HR911105A_C12074
- removed J36, J37, J39: Motor control, Connector_JST:JST_PH_B4B-PH-K_1x04_P2.00mm_Vertical, symbol Connector_Generic:Conn_01x04
- removed L4: 4.7uH, easyeda2kicad:IND-SMD_L7.0-W6.6, symbol Device:L
- removed Q15: SUD50P10-43L-TP, Package_TO_SOT_SMD:TO-252-2, symbol Transistor_FET:SUD50P10-43L
- removed R1, R59, R60, R61, R62, R63, R71, R72, R73, R74: 24, Resistor_SMD:R_2512_6332Metric, symbol Device:R_US
- removed R16, R17, R18: 220, Resistor_SMD:R_2512_6332Metric, symbol Device:R_US
- removed R25: 4.3k, Resistor_SMD:R_1210_3225Metric, symbol Device:R_US
- removed R57, R58: 330, Resistor_SMD:R_0201_0603Metric, symbol Device:R_US
- removed R75: 47k, Resistor_SMD:R_0201_0603Metric, symbol Device:R_US
- removed R76: 10k, Resistor_SMD:R_1206_3216Metric, symbol Device:R_US
- removed R77: 47k T+-1%, Resistor_SMD:R_1206_3216Metric, symbol Device:R_US
- removed R78: 200k, Resistor_SMD:R_0805_2012Metric, symbol Device:R_US
- removed R79: 16k, Resistor_SMD:R_0805_2012Metric, symbol Device:R_US
- removed R80: 120k, Resistor_SMD:R_0805_2012Metric, symbol Device:R_US
- removed R81: 22.1k, Resistor_SMD:R_0805_2012Metric, symbol Device:R_US
- removed RN10, RN11, RN12: 4D03WGJ0102T5E (10k), easyeda2kicad:RES-ARRAY-SMD_0603-8P-L3.2-W1.6-BL, symbol C20197:4D03WGJ0102T5E
- removed RN2, RN3, RN4, RN5: 4D03WGJ0102T5E (1k), easyeda2kicad:RES-ARRAY-SMD_0603-8P-L3.2-W1.6-BL, symbol C20197:4D03WGJ0102T5E
- removed U4: KSZ8081RNAIA-TR, easyeda2kicad:QFN-24_L4.0-W4.0-P0.50-BL-EP2.6, symbol C145623:KSZ8081RNAIA-TR
- removed U6: AP64500SP-13, easyeda2kicad:SOIC-8_L4.9-W3.9-P1.27-LS6.0-BL-EP-1, symbol C2070920:AP64500SP-13
- removed X1: X1G004451000400, easyeda2kicad:OSC-SMD_4P-L5.0-W3.2-BL_SG5032, symbol C37076:X1G004451000400
- added D1: SMF5V0A, Diode_SMD:D_SMF, symbol Diode:SMF5V0A
- added J1, J2, J3: Motor control, Connector_JST:JST_PH_B4B-PH-K_1x04_P2.00mm_Vertical, symbol Connector_Generic:Conn_01x04
- added J4: Screw_Terminal_01x02, easyeda2kicad:CONN-TH_2P-P5.08, symbol Connector:Screw_Terminal_01x02
- added Q2: HSBA100P04_C2987717, easyeda2kicad:DFN-8_L5.7-W5.1-P1.27-LS6.1-BL-1, symbol HSBA100P04:HSBA100P04_C2987717
- added R1: 47k, Resistor_SMD:R_0805_2012Metric, symbol Device:R
- added R10: 4.3k, Resistor_SMD:R_0402_1005Metric, symbol Device:R_US
- added R2: 200k, Resistor_SMD:R_0805_2012Metric, symbol Device:R
- added R3: 16k, Resistor_SMD:R_0805_2012Metric, symbol Device:R
- added R4: 120k, Resistor_SMD:R_0805_2012Metric, symbol Device:R
- added R5: 22.1k, Resistor_SMD:R_0805_2012Metric, symbol Device:R
- added R6: 10k, Resistor_SMD:R_0402_1005Metric, symbol Device:R_US
- added R7, R8, R9: 220, Resistor_SMD:R_0402_1005Metric, symbol Device:R_US
- added U4: AP64500, easyeda2kicad:AP64500SP-13, symbol dcdc-lib:AP64500
- added U6: PCA9685PW,118, easyeda2kicad:TSSOP-28_L9.7-W4.4-P0.65-LS6.4-TL, symbol C2678753_PCA9685PW:PCA9685PW,118
- C1: value 0.1uF -> 10uF; footprint Capacitor_SMD:C_0603_1608Metric -> Capacitor_SMD:C_1206_3216Metric; LCSC https://www.lcsc.com/product-detail/Multilayer-Ceramic-Capa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 -> C13585; LCSC Part C14663 -> (none)
- C2: value 22uF -> 2.7nF; footprint Capacitor_SMD:C_2220_5750Metric -> Capacitor_SMD:C_0805_2012Metric; LCSC C784103 -> C2918070; LCSC Part C784103 -> (none)
- C3: value 2.2uF -> 100nF; footprint Capacitor_SMD:C_2220_5750Metric -> Capacitor_SMD:C_0805_2012Metric; LCSC https://www.lcsc.com/product-detail/Multilayer-Ceramic-Capa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 -> C28233; LCSC Part C23630 -> (none)
- C4: value 0.1uF -> 39pF; footprint Capacitor_SMD:C_0603_1608Metric -> Capacitor_SMD:C_0805_2012Metric; LCSC https://www.lcsc.com/product-detail/Multilayer-Ceramic-Capa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 -> C576897; LCSC Part C14663 -> (none)
- C5: value 22pF -> 47pF; footprint Capacitor_SMD:C_2220_5750Metric -> Capacitor_SMD:C_0805_2012Metric; LCSC https://www.lcsc.com/product-detail/Multilayer-Ceramic-Capa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 -> C113821; LCSC Part C105620 -> (none)
- C6, C8: value 0.1uF -> 22 uF; footprint Capacitor_SMD:C_0603_1608Metric -> Capacitor_SMD:C_1206_3216Metric; LCSC https://www.lcsc.com/product-detail/Multilayer-Ceramic-Capa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 -> C87996; LCSC Part C14663 -> (none)
- C7: value 22uF -> 22 uF; footprint Capacitor_SMD:C_2220_5750Metric -> Capacitor_SMD:C_1206_3216Metric; LCSC C784103 -> C87996; LCSC Part C784103 -> (none)
- C9: value 22uF -> 10uF; footprint Capacitor_SMD:C_2220_5750Metric -> Capacitor_SMD:C_1206_3216Metric; LCSC C784103 -> C13585; LCSC Part C784103 -> (none)
- L1: value BLM21PG331SN1D -> 3.3uH; footprint Inductor_SMD:L_0805_2012Metric -> easyeda2kicad:IND-SMD_L11.6-W10.1; LCSC https://www.lcsc.com/product-detail/Ferrite-Beads_Murata-El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 -> C7587741; LCSC Part C74764 -> (none)
- R15: footprint Resistor_SMD:R_2512_6332Metric -> Resistor_SMD:R_0402_1005Metric; LCSC https://www.lcsc.com/product-detail/Chip-Resistor-Surface-M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 -> (none); LCSC Part C2930459 -> C112291
- R24: footprint Resistor_SMD:R_1210_3225Metric -> Resistor_SMD:R_0402_1005Metric; LCSC https://www.lcsc.com/product-detail/Chip-Resistor-Surface-M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 -> (none); LCSC Part C3000632 -> C112291
- TB1: footprint STM32F4DISCOVERY:MODULE_STM32F4DISCOVERY -> stm32:MODULE_STM32F4DISCOVERY
Connections:
- net Buzzer_Collector is gone; now on net BUZZER_OUT: BUZZER2.2 (-), D7.2 (A)
- net Motor_F_Collector_4 is gone; now on net MOTOR1_FWD: J38.2 (Pin_2)
- net Motor_PWM_Collector_4 is gone; now on net MOTOR1_PWM: J38.1 (Pin_1)
- net Motor_R_Collector_4 is gone; now on net MOTOR1_RVR: J38.3 (Pin_3)
- net VCC (3V) is gone; now on net VCC (5V): R24.1
- net BUZZER_OUT: now also U6.9 (LED3); no longer TB1.P1_24 (PB2)
- net ENC2_A: now also TB1.P2_40 (PA15); no longer TB1.P1_15 (PA5)
- net ENC2_B: now also TB1.P1_11 (PA1); no longer TB1.P2_28 (PB3)
- net ENC3_A: now also TB1.P1_9 (PC3); no longer TB1.P1_18 (PA6)
- net ENC3_B: now also TB1.P2_26 (PB5); no longer TB1.P2_48 (PC7)
- net ETH_CRS_DV: no longer TB1.P1_17 (PA7)
- net ETH_MDC: no longer TB1.P1_7 (PC1)
- net ETH_MDIO: no longer TB1.P1_14 (PA2)
- net ETH_REF_CLK: no longer TB1.P1_11 (PA1)
- net ETH_RXD0: no longer TB1.P1_20 (PC4)
- net ETH_RXD1: no longer TB1.P1_19 (PC5)
- net ETH_TXD0: no longer TB1.P1_36 (PB12)
- net ETH_TXD1: no longer TB1.P1_37 (PB13)
- net ETH_TX_EN: no longer TB1.P1_35 (PB11)
- net GND: now also C1.2, C4.2, C6.2, C8.2, J7.1 (Pin_1), D1.1 (A1), J1.4 (Pin_4), J2.4 (Pin_4), J3.4 (Pin_4), J4.2 (Pin_2), R1.2, R2.2, R5.2, R6.1, U4.7 (GND), U6.1 (A0), U6.14 (VSS), U6.2 (A1), U6.24 (A5), U6.25 (EXTCLK), U6.3 (A2), U6.4 (A3), U6.5 (A4); no longer C1.1, C3.2, C4.1, C5.1, C6.1, C8.1, J7.3 (Pin_3)
- net LED_BLUE_1: now also TB1.P1_37 (PB13); no longer TB1.P2_15 (PE2)
- net LED_BLUE_2: now also TB1.P1_38 (PB14); no longer TB1.P2_16 (PE3)
- net LED_BLUE_3: now also TB1.P1_39 (PB15); no longer TB1.P2_13 (PE4)
- net LED_BLUE_4: now also TB1.P1_36 (PB12); no longer TB1.P2_14 (PE5)
- net LED_Collector_2: now also R7.2
- net LED_Collector_3: now also R8.2
- net LED_Collector_4: now also R9.2
- net LED_GREEN: now also TB1.P1_41 (PD9), U6.15 (LED8); no longer TB1.P1_26 (PE8)
- net LED_RED: now also TB1.P1_43 (PD11), U6.13 (LED7); no longer TB1.P2_11 (PE6)
- net LED_YELLOW: now also TB1.P1_42 (PD10), U6.19 (LED12); no longer TB1.P1_25 (PE7)
- net MOTOR1_FWD: now also U6.7 (LED1); no longer TB1.P1_40 (PD8)
- net MOTOR1_PWM: now also U6.6 (LED0); no longer TB1.P1_34 (PB10)
- net MOTOR1_RVR: now also U6.8 (LED2); no longer TB1.P2_31 (PD3)
- net MOTOR2_FWD: now also J1.2 (Pin_2), U6.11 (LED5); no longer TB1.P1_41 (PD9)
- net MOTOR2_PWM: now also J1.1 (Pin_1), U6.10 (LED4); no longer TB1.P1_13 (PA3)
- net MOTOR2_RVR: now also J1.3 (Pin_3), U6.12 (LED6); no longer TB1.P2_32 (PD4)
- net MOTOR3_FWD: now also J2.2 (Pin_2), U6.21 (LED14); no longer TB1.P1_38 (PB14)
- net MOTOR3_PWM: now also J2.1 (Pin_1), U6.22 (LED15); no longer TB1.P1_22 (PB0)
- net MOTOR3_RVR: now also J2.3 (Pin_3), U6.20 (LED13); no longer TB1.P2_29 (PD5)
- net MOTOR4_FWD: now also J3.2 (Pin_2), U6.17 (LED10); no longer TB1.P1_39 (PB15)
- net MOTOR4_PWM: now also J3.1 (Pin_1), U6.18 (LED11); no longer TB1.P1_21 (PB1)
- net MOTOR4_RVR: now also J3.3 (Pin_3), U6.16 (LED9); no longer TB1.P2_30 (PD6)
- net POWER_SUPPLY_ADC: now also TB1.P1_7 (PC1); no longer TB1.P1_16 (PA4)
- net TTL_RX: now also J7.3 (Pin_3); no longer J7.1 (Pin_1), TB1.P2_38 (PC11)
- net TTL_TX: no longer TB1.P1_12 (PA0-WKUP)
- net US_SENSOR1_TRIG: now also TB1.P1_30 (PE12); no longer TB1.P1_42 (PD10)
- net US_SENSOR2_TRIG: now also TB1.P1_33 (PE15); no longer TB1.P1_43 (PD11)
- net VCC (5V): now also C5.1, C6.1, C7.1, C8.1, C9.1, L1.2, D1.2 (A2), J4.1 (Pin_1), Q2.5 (D), R10.1, R4.1, U6.28 (VDD)
- net at U7.2 (K): now also R9.1
- net at C3.1: now also U4.1 (BST); no longer C1.2
- net at U3.2 (K): now also R8.1
- net at C5.2: now also R4.2, R5.1, U4.5 (FB)
- net at C2.1: now also R3.2; no longer C4.2
- net at U2.2 (K): now also R7.1
- net SDA: now reaches TB1.P2_44 (PA9)
- net SDA: now also J11.1 (Pin_1), R24.2, U5.24 (SDA), U6.27 (SDA)
- net COMPASS_SCL: no longer names the net of TB1.P2_23 (PB6)
- net COMPASS_SCL: no longer J11.2 (Pin_2)
- removed net COMPASS_SDA: J11.1 (Pin_1), R24.2, TB1.P2_24 (PB7)
- net GPS_RX: no longer names the net of TB1.P2_34 (PD2)
- net GPS_TX: no longer names the net of TB1.P2_35 (PC12)
- net MPU_SCL renamed SCL
- net SCL: now also J11.2 (Pin_2), R10.2, U6.26 (SCL)
- net MPU_SDA: no longer names the net of TB1.P2_46 (PC9)
- net MPU_SDA: no longer U5.24 (SDA)
- removed net VCC (3.3V): C8.2, C9.1, L1.1
- new net: C1.1, Q2.1 (S), Q2.2 (S), Q2.3 (S), U4.2 (VIN), U4.3 (EN)
- new net: Q2.4 (G), R1.1
- new net: R6.2, U6.23 (~{OE})
- new net: C3.2, L1.1, U4.8 (SW)
- new net: C4.1, R3.1, U4.6 (COMP)
- new net: R2.1, U4.4 (RT/CLK)
Other:
- removed sheet transistor_array
- removed sheet transistor_array1
- removed sheet transistor_array2
- removed sheet transistor_array3
- note added: "External PWM driver"
- note added: "Screw Connector Input"
- note removed: "Ethernet transreciever"
- note removed: "GPS Interface"
- note removed: "Transistors Connections (4X)"
- note removed: "actually, i don't quite understand how to choose suitable ferrite bead. i chose one that is equal to Ethernet frequency and has high impedance. i guess, later, we should replace it with a more suitable. later is when i will properly read the documentation."
- note removed: "add lcsc links"
- note removed: "also, connect paddle to the GND."
- note removed: "collector has two pins for better current handling and thermal dissipation"
- note removed: "here, we can connect OE/ST to the VCC to enable crystal constantly. or control it with XO."
- note removed: "maybe it needs to be connected to the GND"
- note removed: "special pin in open-drain mode."
- note removed: "the pins will be populated later. when we will know what we need. Andrii is dealing with this."
- moved on the sheet: BUZZER2, C100, C101, C102, C11, C15, C19, C20, C33, C34, C73, C95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
