File: rover-chasis-controller.kicad_sch (KiCad schematic)
At the start: 78 parts, among them J1 Motor control, J11 Compass Connection (I2C), J15 External LED (Red), J16 External LED (Yellow), J17 External LED (Green), J2 Motor control, J22 Ultrasonic Sensor Inputs, J3 Motor control, J38 Motor control, J4 Screw_Terminal_01x02, J40 Encoder, J41 Encoder, J42 Encoder, J43 Encoder, J7 TTL, J8 Ultrasonic Sensor Inputs, Q2 HSBA100P04_C2987717, U1 APT2012LVBC/D, U2 APT2012LVBC/D, U3 APT2012LVBC/D, U4 AP64500, U5 MPU-6050_C24112, U6 PCA9685PW,118, U7 APT2012LVBC/D

Commit message: Issue #1: Replaced out-of-stock components
Parts:
- J1, J11, J2, J22, J3, J38, J40, J41, J42, J43, J8: LCSC Part C111514 -> C131334
- J15, J16, J17: LCSC Part C495693 -> C131337
- J7: LCSC Part C265393 -> C131339
- U1, U2, U3, U7: footprint easyeda2kicad:LED-SMD_L2.0-W1.3-R-RD -> LED_SMD:LED_0805_2012Metric; LCSC Part C5879383 -> C965817

Commit message: Issue #1: Removed unnecessary fields inside components
Parts:
- C1, C9: LCSC C13585 -> (none)
- C10, C100, C101, C102, C19, C20, C33, C73, C95, C96, C97, C98, C99: LCSC https://www.lcsc.com/product-detail/Multilayer-Ceramic-Capa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 -> (none)
- C2: LCSC C2918070 -> (none)
- C3: LCSC C28233 -> (none)
- C4: LCSC C576897 -> (none)
- C5: LCSC C113821 -> (none)
- C6, C7, C8: LCSC C87996 -> (none)
- F1, F2, F3, F9: LCSC https://www.lcsc.com/product-detail/Resettable-Fuses_BNstar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 -> (none)
- J1, J11, J2, J22, J3, J38, J40, J41, J42, J43, J8: LCSC https://www.lcsc.com/product-detail/Housings-Wire-To-Board-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 -> (none)
- L1: LCSC C7587741 -> (none)
- R1: LCSC C2989281 -> (none)
- R2: LCSC C728645 -> (none)
- RN1: LCSC https://www.lcsc.com/product-detail/Resistor-Networks-Array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 -> (none)
Changed lines of the file:
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@@
 			)
 		)
-		(property "LCSC" "https://www.lcsc.com/product-detail/Multilayer-Ceramic-Capacitors-MLCC-SMD-SMT_YAGEO-CC0603KRX7R9BB104_C14663.html?s_z=n_100nf%2520smd"
+		(property "LCSC" ""
 			(at 158.75 135.89 90)
 			(effects
@@
 			)
 		)
-		(property "LCSC" "https://www.lcsc.com/product-detail/Resettable-Fuses_BNstar-SMD1812-030C-30V_C2760284.html?s_z=n_smd%2520fuse%25200.3A"
+		(property "LCSC" ""
 			(at 316.23 102.87 90)
 			(effects
@@
 			)
 		)
-		(property "LCSC" "https://www.lcsc.com/product-detail/Multilayer-Ceramic-Capacitors-MLCC-SMD-SMT_YAGEO-CC0603KRX7R9BB104_C14663.html?s_z=n_100nf%2520smd"
+		(property "LCSC" ""
 			(at 331.47 106.68 90)
 			(effects
@@
 			)
 		)
-		(property "LCSC" "https://www.lcsc.com/product-detail/Multilayer-Ceramic-Capacitors-MLCC-SMD-SMT_YAGEO-CC0603KRX7R9BB104_C14663.html?s_z=n_100nf%2520smd"
+		(property "LCSC" ""
 			(at 331.47 129.54 90)
 			(effects
@@
 			)
 		)
-		(property "LCSC" "https://www.lcsc.com/product-detail/Housings-Wire-To-Board-Wire-To-Wire_JST-PHR-4_C111514.html?s_z=n_jst%20ph%204"
+		(property "LCSC" ""
 			(at 191.77 200.66 0)
 			(effects
@@
 			)
 		)
-		(property "LCSC" "C87996"
+		(property "LCSC" ""
 			(at 231.775 51.435 0)
 			(effects
@@
 			)
 		)
-		(property "LCSC" "https://www.lcsc.com/product-detail/Housings-Wire-To-Board-Wire-To-Wire_JST-PHR-4_C111514.html?s_z=n_jst%20ph%204"
+		(property "LCSC" ""
 			(at 264.16 154.94 0)
 			(effects
@@
 			)
 		)
-		(property "LCSC" "C2918070"
+		(property "LCSC" ""
 			(at 172.085 74.295 0)
 			(effects
@@
 			)
 		)
-		(property "LCSC" "https://www.lcsc.com/product-detail/Multilayer-Ceramic-Capacitors-MLCC-SMD-SMT_YAGEO-CC0603KRX7R9BB104_C14663.html?s_z=n_100nf%2520smd"
+		(property "LCSC" ""
 			(at 102.87 238.76 90)
 			(effects
@@
 			)
 		)
-		(property "LCSC" "https://www.lcsc.com/product-detail/Housings-Wire-To-Board-Wire-To-Wire_JST-PHR-4_C111514.html?s_z=n_jst%20ph%204"
+		(property "LCSC" ""
 			(at 306.07 100.33 0)
 			(effects
@@
 			)
 		)
-		(property "LCSC" "C7587741"
+		(property "LCSC" ""
 			(at 184.15 41.91 90)
 			(effects
@@
 			)
 		)
-		(property "LCSC" "C113821"
+		(property "LCSC" ""
 			(at 193.04 45.72 0)
 			(effects
@@
 			)
 		)
-		(property "LCSC" "https://www.lcsc.com/product-detail/Housings-Wire-To-Board-Wire-To-Wire_JST-PHR-4_C111514.html?s_z=n_jst%20ph%204"
+		(property "LCSC" ""
 			(at 138.43 210.82 0)
 			(effects
@@
 			)
 		)
-		(property "LCSC" "https://www.lcsc.com/product-detail/Housings-Wire-To-Board-Wire-To-Wire_JST-PHR-4_C111514.html?s_z=n_jst%20ph%204"
+		(property "LCSC" ""
 			(at 245.11 222.25 0)
 			(effects
@@
 			)
 		)
-		(property "LCSC" "https://www.lcsc.com/product-detail/Multilayer-Ceramic-Capacitors-MLCC-SMD-SMT_Samsung-Electro-Mechanics-CL21A106KOQNNNE_C1713.html?s_z=n_10uF%2520smd"
+		(property "LCSC" ""
 			(at 275.59 129.54 90)
 			(effects
@@
 			)
 		)
-		(property "LCSC" "C87996"
+		(property "LCSC" ""
 			(at 224.79 51.435 0)
 			(effects
@@
 			)
 		)
-		(property "LCSC" "https://www.lcsc.com/product-detail/Multilayer-Ceramic-Capacitors-MLCC-SMD-SMT_Samsung-Electro-Mechanics-CL21A106KOQNNNE_C1713.html?s_z=n_10uF%2520smd"
+		(property "LCSC" ""
 			(at 275.59 106.68 90)
 			(effects
@@
 			)
 		)
-		(property "LCSC" "https://www.lcsc.com/product-detail/Multilayer-Ceramic-Capacitors-MLCC-SMD-SMT_YAGEO-CC0603KRX7R9BB104_C14663.html?s_z=n_100nf%2520smd"
+		(property "LCSC" ""
 			(at 149.86 217.17 90)
 			(effects
@@
 			)
 		)
-		(property "LCSC" "https://www.lcsc.com/product-detail/Multilayer-Ceramic-Capacitors-MLCC-SMD-SMT_YAGEO-CC0603KRX7R9BB104_C14663.html?s_z=n_100nf%2520smd"
+		(property "LCSC" ""
 			(at 284.48 129.54 90)
 			(effects
@@
 			)
 		)
-		(property "LCSC" "https://www.lcsc.com/product-detail/Resettable-Fuses_BNstar-SMD1812-030C-30V_C2760284.html?s_z=n_smd%2520fuse%25200.3A"
+		(property "LCSC" ""
 			(at 269.24 102.87 90)
 			(effects
@@
 			)
 		)
-		(property "LCSC" "C2989281"
+		(property "LCSC" ""
 			(at 116.84 52.07 0)
 			(effects
@@
 			)
 		)
-		(property "LCSC" "https://www.lcsc.com/product-detail/Multilayer-Ceramic-Capacitors-MLCC-SMD-SMT_YAGEO-CC0603KRX7R9BB104_C14663.html?s_z=n_100nf%2520smd"
+		(property "LCSC" ""
 			(at 284.48 106.68 90)
 			(effects
@@
 			)
 		)
-		(property "LCSC" "https://www.lcsc.com/product-detail/Multilayer-Ceramic-Capacitors-MLCC-SMD-SMT_Samsung-Electro-Mechanics-CL21A106KOQNNNE_C1713.html?s_z=n_10uF%2520smd"
+		(property "LCSC" ""
 			(at 322.58 129.54 90)
 			(effects
@@
 			)
 		)
-		(property "LCSC" "C13585 "
+		(property "LCSC" ""
 			(at 130.175 46.355 0)
 			(effects
@@
 			)
 		)
-		(property "LCSC" "C576897"
+		(property "LCSC" ""
 			(at 184.15 64.77 0)
 			(effects
@@
 			)
 		)
-		(property "LCSC" "https://www.lcsc.com/product-detail/Resettable-Fuses_BNstar-SMD1812-030C-30V_C2760284.html?s_z=n_smd%2520fuse%25200.3A"
+		(property "LCSC" ""
 			(at 316.23 125.73 90)
 			(effects
@@
 			)
 		)
-		(property "LCSC" "https://www.lcsc.com/product-detail/Multilayer-Ceramic-Capacitors-MLCC-SMD-SMT_Samsung-Electro-Mechanics-CL21A106KOQNNNE_C1713.html?s_z=n_10uF%2520smd"
+		(property "LCSC" ""
 			(at 156.21 217.17 90)
 			(effects
@@
 			)
 		)
-		(property "LCSC" "https://www.lcsc.com/product-detail/Multilayer-Ceramic-Capacitors-MLCC-SMD-SMT_YAGEO-CC0603KRX7R9BB104_C14663.html?s_z=n_100nf%2520smd"
+		(property "LCSC" ""
 			(at 280.67 161.29 90)
 			(effects
@@
 			)
 		)
-		(property "LCSC" "https://www.lcsc.com/product-detail/Housings-Wire-To-Board-Wire-To-Wire_JST-PHR-4_C111514.html?s_z=n_jst%20ph%204"
+		(property "LCSC" ""
 			(at 276.86 199.39 0)
 			(effects
@@
 			)
 		)
-		(property "LCSC" "https://www.lcsc.com/product-detail/Housings-Wire-To-Board-Wire-To-Wire_JST-PHR-4_C111514.html?s_z=n_jst%20ph%204"
+		(property "LCSC" ""
 			(at 259.08 123.19 0)
 			(effects
@@
 			)
 		)
-		(property "LCSC" "C87996"
+		(property "LCSC" ""
 			(at 216.535 51.435 0)
 			(effects
@@
 			)
 		)
-		(property "LCSC" "C728645"
+		(property "LCSC" ""
 			(at 138.43 63.5 0)
 			(effects
@@
 			)
 		)
-		(property "LCSC" "C28233"
+		(property "LCSC" ""
 			(at 176.53 36.83 0)
 			(effects
@@
 			)
 		)
-		(property "LCSC" "https://www.lcsc.com/product-detail/Resistor-Networks-Arrays_UNI-ROYAL-Uniroyal-Elec-4D03WGJ0102T5E_C20197.html?s_z=s_Resistors%257CResistor%2520Networks%252C%2520Arrays"
+		(property "LCSC" ""
 			(at 198.12 160.02 0)
 			(effects
@@
 			)
 		)
-		(property "LCSC" "https://www.lcsc.com/product-detail/Housings-Wire-To-Board-Wire-To-Wire_JST-PHR-4_C111514.html?s_z=n_jst%20ph%204"
+		(property "LCSC" ""
 			(at 276.86 222.25 0)
 			(effects
@@
 			)
 		)
-		(property "LCSC" "C13585 "
+		(property "LCSC" ""
 			(at 307.34 38.1 0)
 			(effects
@@
 			)
 		)
-		(property "LCSC" "https://www.lcsc.com/product-detail/Resettable-Fuses_BNstar-SMD1812-030C-30V_C2760284.html?s_z=n_smd%2520fuse%25200.3A"
+		(property "LCSC" ""
 			(at 269.24 125.73 90)
 			(effects
@@
 			)
 		)
-		(property "LCSC" "https://www.lcsc.com/product-detail/Housings-Wire-To-Board-Wire-To-Wire_JST-PHR-4_C111514.html?s_z=n_jst%20ph%204"
+		(property "LCSC" ""
 			(at 259.08 100.33 0)
 			(effects
@@
 			)
 		)
-		(property "LCSC" "https://www.lcsc.com/product-detail/Housings-Wire-To-Board-Wire-To-Wire_JST-PHR-4_C111514.html?s_z=n_jst%20ph%204"
+		(property "LCSC" ""
 			(at 306.07 123.19 0)
 			(effects
@@
 			)
 		)
-		(property "LCSC" "https://www.lcsc.com/product-detail/Multilayer-Ceramic-Capacitors-MLCC-SMD-SMT_Samsung-Electro-Mechanics-CL21A106KOQNNNE_C1713.html?s_z=n_10uF%2520smd"
+		(property "LCSC" ""
 			(at 322.58 106.68 90)
 			(effects
@@
 			)
 		)
-		(property "LCSC" "https://www.lcsc.com/product-detail/Housings-Wire-To-Board-Wire-To-Wire_JST-PHR-4_C111514.html?s_z=n_jst%20ph%204"
+		(property "LCSC" ""
 			(at 245.11 200.66 0)
 			(effects

Commit message: Board malfunction fixes
- Changed F1-F4, R5, R6 to 3V (previous 5V caused failure).

- Connected STM32DISC1 to 5V and 3V outputs/inputs

- Moved SDA to PC9 (was PA9) and ENC3_A to PC6 (was PC3).

- Redesigned MPU6050 layout to resolve stability and connectivity issues.

- Isolated PCA6587 buzzer with a transistor.
Parts:
- removed U2, U3, U7: APT2012LVBC/D, LED_SMD:LED_0805_2012Metric, symbol C5879383:APT2012LVBC_D
- added C26: 10nF, Capacitor_SMD:C_0402_1005Metric, symbol Device:C
- added J17, J32: Conn_02x25_Counter_Clockwise, symbol Connector_Generic:Conn_02x25_Counter_Clockwise
- added J18, J19, J20, J21, J22, J27, J28, J29, J30, J31: Conn_01x04, symbol Connector_Generic:Conn_01x04
- added J23: Conn_01x03, symbol Connector_Generic:Conn_01x03
- added J24, J25, J26: Conn_01x02, symbol Connector_Generic:Conn_01x02
- added Q6: MMBT3904_C181119, easyeda2kicad:SOT-23-3_L2.9-W1.6-P1.90-LS2.8-BR, symbol C181119:MMBT3904_C181119
- added R15: 1k, Resistor_SMD:R_0402_1005Metric, symbol Device:R_US
- added U4, U5, U6: APT2012LVBC/D, easyeda2kicad:LED-SMD_L2.0-W1.3-R-RD, symbol C5879383:APT2012LVBC_D
- C1: renamed from C10; LCSC (none) -> https://www.lcsc.com/product-detail/Multilayer-Ceramic-Capa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
- C10: renamed from C4; LCSC (none) -> C576897
- C11: renamed from C5; LCSC (none) -> C113821
- C13: renamed from C6; LCSC (none) -> C87996
- C14: renamed from C7; LCSC (none) -> C87996
- C15: renamed from C8; LCSC (none) -> C87996
- C16: renamed from C95; value 10uF -> 10uFx16V; LCSC (none) -> https://www.lcsc.com/product-detail/Multilayer-Ceramic-Capa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; LCSC Part C1713 -> C18185764
- C17: renamed from C101; value 10uF -> 10uFx16V; LCSC (none) -> https://www.lcsc.com/product-detail/Multilayer-Ceramic-Capa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; LCSC Part C1713 -> C18185764
- C18: renamed from C73; LCSC (none) -> https://www.lcsc.com/product-detail/Multilayer-Ceramic-Capa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
- C19: renamed from C97; LCSC (none) -> https://www.lcsc.com/product-detail/Multilayer-Ceramic-Capa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
- C20: renamed from C102; LCSC (none) -> https://www.lcsc.com/product-detail/Multilayer-Ceramic-Capa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
- C21: renamed from C9; value 10uF -> 10uFx16V; footprint Capacitor_SMD:C_1206_3216Metric -> Capacitor_SMD:C_0805_2012Metric; LCSC (none) -> C18185764; LCSC Part C1713 -> C18185764
- C22: renamed from C96; value 10uF -> 10uFx16V; LCSC (none) -> https://www.lcsc.com/product-detail/Multilayer-Ceramic-Capa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; LCSC Part C1713 -> C18185764
- C23: renamed from C99; value 10uF -> 10uFx16V; LCSC (none) -> https://www.lcsc.com/product-detail/Multilayer-Ceramic-Capa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; LCSC Part C1713 -> C18185764
- C24: renamed from C98; LCSC (none) -> https://www.lcsc.com/product-detail/Multilayer-Ceramic-Capa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
- C25: renamed from C100; LCSC (none) -> https://www.lcsc.com/product-detail/Multilayer-Ceramic-Capa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
- C3: renamed from C1; value 10uF -> 10uFx50V; LCSC (none) -> C513774; LCSC Part C1713 -> C513774
- C4: renamed from C20; LCSC (none) -> https://www.lcsc.com/product-detail/Multilayer-Ceramic-Capa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
- C5: renamed from C19; value 10uF -> 10uFx16V; LCSC (none) -> https://www.lcsc.com/product-detail/Multilayer-Ceramic-Capa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; LCSC Part C1713 -> C18185764
- C6: renamed from C33; LCSC (none) -> https://www.lcsc.com/product-detail/Multilayer-Ceramic-Capa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
- C7: renamed from C34; LCSC Part C28260 -> C107146
- C8: renamed from C2; LCSC (none) -> C2918070
- C9: renamed from C3; LCSC (none) -> C28233
- F1: renamed from F9; LCSC (none) -> https://www.lcsc.com/product-detail/Resettable-Fuses_BNstar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
- F2: renamed from F3; LCSC (none) -> https://www.lcsc.com/product-detail/Resettable-Fuses_BNstar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
- F3: renamed from F1; LCSC (none) -> https://www.lcsc.com/product-detail/Resettable-Fuses_BNstar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
- F4: renamed from F2; LCSC (none) -> https://www.lcsc.com/product-detail/Resettable-Fuses_BNstar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
- J10: renamed from J40; LCSC (none) -> https://www.lcsc.com/product-detail/Housings-Wire-To-Board-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
- J11: renamed from J43; LCSC (none) -> https://www.lcsc.com/product-detail/Housings-Wire-To-Board-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
- J12: renamed from J22; LCSC (none) -> https://www.lcsc.com/product-detail/Housings-Wire-To-Board-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
- J13: renamed from J1; LCSC (none) -> https://www.lcsc.com/product-detail/Housings-Wire-To-Board-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
- J14: renamed from J3; LCSC (none) -> https://www.lcsc.com/product-detail/Housings-Wire-To-Board-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
- J15: renamed from J41; LCSC (none) -> https://www.lcsc.com/product-detail/Housings-Wire-To-Board-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
- J16: renamed from J42; LCSC (none) -> https://www.lcsc.com/product-detail/Housings-Wire-To-Board-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
- J5: renamed from J11; LCSC (none) -> https://www.lcsc.com/product-detail/Housings-Wire-To-Board-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
- J7: renamed from J8; LCSC (none) -> https://www.lcsc.com/product-detail/Housings-Wire-To-Board-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
- J8: renamed from J38; LCSC (none) -> https://www.lcsc.com/product-detail/Housings-Wire-To-Board-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
- J9: renamed from J2; LCSC (none) -> https://www.lcsc.com/product-detail/Housings-Wire-To-Board-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
- L1: LCSC (none) -> C7587741
- R3: renamed from R1; LCSC (none) -> C2989281
- R4: renamed from R2; LCSC (none) -> C728645
- R5: renamed from R24; footprint Resistor_SMD:R_1206_3216Metric -> Resistor_SMD:R_0805_2012Metric; LCSC Part C2933704 -> C728653
- R6: renamed from R10; footprint Resistor_SMD:R_1206_3216Metric -> Resistor_SMD:R_0805_2012Metric; LCSC Part C2933704 -> C728653
- RN1: LCSC (none) -> https://www.lcsc.com/product-detail/Resistor-Networks-Array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
- TB1: LCSC Part C118360 -> (none)
- U3: renamed from U1; footprint LED_SMD:LED_0805_2012Metric -> easyeda2kicad:LED-SMD_L2.0-W1.3-R-RD
- renumbered BUZZER2 to BUZZER1, C15 to C12, C11 to C2, D7 to D1, D1 to D2, J17 to J1, J16 to J2, J15 to J3, J7 to J6, MK5 to MK1, MK1 to MK2, MK2 to MK3, MK3 to MK4, MK4 to MK5, Q2 to Q1, R11 to R1, R15 to R10, R7 to R11, R8 to R12, R9 to R13, R6 to R14, R12 to R2, R3 to R7, R4 to R8, R5 to R9, U5 to U1, U4 to U2, U6 to U7
Connections:
- net BUZZER_OUT: now also R15.1; no longer BUZZER1.2 (-), D1.2 (A)
- net ENC3_A: now also TB1.P2_47 (PC6); no longer TB1.P1_9 (PC3)
- net GND: now also U1.9 (AD0), C26.1, Q6.2
- net SDA: now also TB1.P2_46 (PC9); no longer TB1.P2_44 (PA9)
- net VCC (5V): now also TB1.P2_3 (5V), TB1.P2_4 (5V), U4.1 (A), U5.1 (A), U6.1 (A); no longer C16.2, C17.2, C19.2, C20.2, C22.2, C23.2, C24.2, C25.2, F1.2, F2.2, F3.2, F4.2, R5.1, R6.1
- net VDD (3V): now also C16.2, C17.2, C19.2, C20.2, C22.2, C23.2, C24.2, C25.2, F1.2, F2.2, F3.2, F4.2, R5.1, R6.1, TB1.P2_5 (3V), TB1.P2_6 (3V), U1.8 (VLOGIC), C26.2
- net at R13.1: now also U6.2 (K)
- net at R11.1: now also U4.2 (K)
- net at R12.1: now also U5.2 (K)
- new net: Q6.1, R15.2
- new net: BUZZER1.2 (-), D1.2 (A), Q6.3
Other:
- note added: "0x68"
- note removed: "TODO: 7. Resolve all ERC exceptions and warnings. 9. Recalculate all of the numerical values for scheme, to be sure. 13. Consider implement Multi unit symbols for IC Arrays. 15. Include PWR_FLAG, properly. DONE: 1. Rework transisor schemes with transistor arrays. 1.1 Motor controllers. 1.2 External LEDs. 1.3 Buzzer. 2. Rework power supply by taking already in use PMIC in rpi-power-HAT. (Varya PCB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"
- note removed: "Коли використовувати VLOGIC: Якщо ви підключаєте MPU-6050 до мікроконтролера, який працює на логічних рівнях 1.8В або 5В, тоді ви можете використовувати VLOGIC для встановлення рівнів логіки, сумісних із мікроконтролером. VLOGIC дозволяє забезпечити сумісність між рівнями сигналів I2C (SDA/SCL) і рівнями GPIO мікроконтролера. Коли можна обійтися без VLOGIC: Якщо ваш STM32 працює на 3.3В, як і сам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"
- company: (none) -> KPI Rover
- title: Rover Chassis Controller PCB -> Chassis Controller
- moved on the sheet: BUZZER1, C1, C12, C4, C5, D1, J13, J14, J4, J5, J6, J7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
