File: chassis_controller.kicad_sch (KiCad schematic)
At the start: 128 parts, among them J1 Screw_Terminal_01x02, J10 Conn_01x04_Pin, J11 Conn_02x03_Odd_Even, J12 Conn_01x04_Pin, J13 Conn_01x04_Pin, J14 Conn_01x04_Pin, J15 Conn_01x04_Pin, J16 Conn_01x04_Pin, J17 Conn_01x04_Pin, J18 Conn_01x03_Pin, J19 Conn_01x03_Pin, J2 Conn_01x04_Pin, J20 Conn_01x03_Pin, J21 Conn_01x04_Pin, J22 Conn_01x03_Pin, J23 Conn_01x03_Pin, J24 Conn_01x03_Pin, J25 Conn_01x03_Pin, J3 Conn_01x02_Pin, J4 Conn_01x02_Pin, J5 Conn_01x03_Pin, J6 Conn_01x03_Pin, J7 Conn_01x04_Pin, J8 Conn_01x04_Pin, J9 Conn_01x04_Pin, Q2 HSBA100P04, Q4 HSBA100P04, U1 AP64500SP-13, U2 AMS1117-3.3, U3 DSHP04TSGER, U4 STM32F407VGT6TR, U5 PCA9685PW,118, U6 PCA9685PW,118, U7 MPU-6050, U8 SN65HVD230DR, X1 X32258MOB4SI

Commit message: Add improvements to project
Parts:
- removed J11: Conn_02x03_Odd_Even, Connector_IDC:IDC-Header_2x03_P2.54mm_Vertical, symbol Connector_Generic:Conn_02x03_Odd_Even
- added C46, C47: 1000uF, Capacitor_THT:CP_Radial_D10.0mm_P5.00mm, symbol Device:C_Polarized
- added J26: Conn_01x06_Pin, Connector_JST:JST_PH_B6B-PH-K_1x06_P2.00mm_Vertical, symbol Connector:Conn_01x06_Pin
- added Q1: NMOS, Package_TO_SOT_SMD:SOT-23, symbol Simulation_SPICE:NMOS
- added R16: 47k, Resistor_SMD:R_0805_2012Metric, symbol Device:R
- R19: value 10 -> 10k; LCSC Part C865142 -> C110775
Connections:
- net +3.3V: now also J26.1 (Pin_1)
- net GND: now also R19.2, X1.2 (GND), C46.2, C47.2, J26.3 (Pin_3), Q1.3 (S); no longer X1.3
- net MOTOR1_FWD: now also U5.11 (LED5); no longer U5.10 (LED4)
- net MOTOR1_PWM: now also U5.10 (LED4); no longer U4.61 (PD14)
- net MOTOR1_RVR: now also U5.12 (LED6); no longer U5.11 (LED5)
- net MOTOR2_FWD: now also U5.15 (LED8); no longer U5.12 (LED6)
- net MOTOR2_PWM: now also U5.13 (LED7); no longer U4.62 (PD15)
- net MOTOR2_RVR: now also U5.16 (LED9); no longer U5.13 (LED7)
- net MOTOR3_FWD: now also U5.18 (LED11); no longer U5.15 (LED8)
- net MOTOR3_PWM: now also U5.17 (LED10); no longer U4.25 (PA2)
- net MOTOR3_RVR: now also U5.19 (LED12); no longer U5.16 (LED9)
- net MOTOR4_FWD: now also U5.21 (LED14); no longer U5.17 (LED10)
- net MOTOR4_PWM: now also U5.20 (LED13); no longer U4.26 (PA3)
- net MOTOR4_RVR: now also U5.22 (LED15); no longer U5.18 (LED11)
- net NRST: now also J26.5 (Pin_5)
- net OSC_IN: now also X1.3; no longer X1.2 (GND)
- net SERVO_5V: now also C46.1, C47.1
- net SERVO_PWR: now also R16.1; no longer R19.1
- net SWCLK: now also J26.2 (Pin_2)
- net SWDIO: now also J26.4 (Pin_4)
- net SWO: now also J26.6 (Pin_6)
- net at Q4.4 (G), R18.2: now also Q1.1 (D); no longer R19.2
- new net: Q1.2 (G), R16.2, R19.1
Other:
- moved on the sheet: Q4, R18, R22, R23, R24, R25, R32, U3

Commit message: Update project
Parts:
- removed C39: 10nF, Capacitor_SMD:C_0805_2012Metric, symbol Device:C
- removed C46: 1000uF, Capacitor_THT:CP_Radial_D10.0mm_P5.00mm, symbol Device:C_Polarized
- removed J3: Conn_01x02_Pin, Connector_JST:JST_PH_B2B-PH-K_1x02_P2.00mm_Vertical, symbol Connector:Conn_01x02_Pin
- added C46: 100nF, Capacitor_SMD:C_0805_2012Metric, symbol Device:C
- added C48: 1000uF, Capacitor_THT:CP_Radial_D10.0mm_P5.00mm, symbol Device:C_Polarized
- added J3: Screw_Terminal_01x02, DB127V-5.08-2P-GN-S:CONN-TH_2P-P5.08, symbol Connector:Screw_Terminal_01x02
- added Q3: NMOS, Package_TO_SOT_SMD:SOT-23, symbol Simulation_SPICE:NMOS
- added R36, R37: 4.7k, Resistor_SMD:R_0805_2012Metric, symbol Device:R
- added R38, R39, R40, R46, R47, R48, R49, R50, R51, R52: 0, Resistor_SMD:R_0805_2012Metric, symbol Device:R
- added R41: 330, Resistor_SMD:R_0805_2012Metric, symbol Device:R
- added R42, R43: 1k, Resistor_SMD:R_0805_2012Metric, symbol Device:R
- added R44, R45: 2k, Resistor_SMD:R_0805_2012Metric, symbol Device:R
- Q1: LCSC Part C16338 -> C347475
Connections:
- net +3.3V: now also R40.1, R49.1, R50.2, R51.2, R52.1, R52.2; no longer C43.1, R22.1, R23.1, R24.1, R25.1, R30.1, R31.1, U7.13 (VDD), U7.8 (VLOGIC), U8.3 (VCC)
- net +5V: now also C47.1, C48.1, J3.1 (Pin_1), R38.1, R39.1, R46.1, R47.1, R48.1; no longer BUZZER1.1, C15.1, C36.1, C37.1, R1.2, R11.2, R28.1, R29.1, R4.2, R7.2, U2.3 (VIN), U5.28 (VDD), U6.28 (VDD)
- net BUZZER_OUT: now also R41.2; no longer BUZZER1.2
- net GND: now also U7.9 (AD0), C46.1, C48.2, J3.2 (Pin_2), Q3.3 (S), R44.2, R45.2; no longer U5.1 (A0), U6.2 (A1)
- net SERVO_5V: no longer C47.1
- net USS1_ECHO: now also R42.1, R44.1; no longer J14.4 (Pin_4)
- net USS2_ECHO: now also R43.1, R45.1; no longer J15.4 (Pin_4)
- new net: R1.2, R11.2, R4.2, R48.2, R7.2
- new net: C43.1, C46.2, R30.1, R31.1, R49.2, U7.13 (VDD), U7.8 (VLOGIC)
- new net: R36.2, U5.1 (A0)
- new net: C36.1, R36.1, R38.2, U5.28 (VDD)
- new net: R28.1, R29.1, R50.1
- new net: BUZZER1.1, R46.2
- new net: BUZZER1.2, Q3.1 (D)
- new net: C37.1, R37.1, R39.2, U6.28 (VDD)
- new net: R37.2, U6.2 (A1)
- new net: R22.1, R23.1, R24.1, R25.1, R51.1
- new net: J15.4 (Pin_4), R43.2
- new net: R40.2, U8.3 (VCC)
- new net: C15.1, R47.2, U2.3 (VIN)
- new net: J14.4 (Pin_4), R42.2
- new net: Q3.2 (G), R41.1
- no-connect marks 69 -> 68
Other:
- moved on the sheet: BUZZER1, C24, C25, C26, C27, C42, C47, D1, D4, D5, D6, J14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
